Commit message: All hooked up

File: src/cmr_description/cmr_drives_description/ros2_control/drives.ros2_control.xacro (robot description, xacro)
@@ -6,10 +6,30 @@
                 <plugin>cmr_control/DrivesSystemHardware</plugin>
             </hardware>
-            <joint name="left_wheel_joint">
+            <joint name="left_front_joint">
                 <command_interface name="velocity"/>
                 <state_interface name="position"/>
                 <state_interface name="velocity"/>
             </joint>
-            <joint name="right_wheel_joint">
+            <joint name="left_mid_joint">
+                <command_interface name="velocity"/>
+                <state_interface name="position"/>
+                <state_interface name="velocity"/>
+            </joint>
+            <joint name="left_back_joint">
+                <command_interface name="velocity"/>
+                <state_interface name="position"/>
+                <state_interface name="velocity"/>
+            </joint>
+            <joint name="right_front_joint">
+                <command_interface name="velocity"/>
+                <state_interface name="position"/>
+                <state_interface name="velocity"/>
+            </joint>
+            <joint name="right_mid_joint">
+                <command_interface name="velocity"/>
+                <state_interface name="position"/>
+                <state_interface name="velocity"/>
+            </joint>
+            <joint name="right_back_joint">
                 <command_interface name="velocity"/>
                 <state_interface name="position"/>

File: src/cmr_description/cmr_drives_description/urdf/drives.urdf.xacro (robot description, xacro)
@@ -8,3 +8,4 @@
     <xacro:include filename="$(find cmr_drives_description)/ros2_control/drives.ros2_control.xacro" />
     <xacro:drives />
+    <xacro:drives_ros2_control name="drives"/>
 </robot>

File: src/cmr_description/cmr_drives_description/urdf/drives_description.urdf.xacro (robot description, xacro)
@@ -13,9 +13,35 @@
         <xacro:property name="wheel_len" value="0.020" />
         <xacro:property name="wheel_radius" value="0.015" />
-        <xacro:property name="caster_wheel_mass" value="0.1" />
-        <!-- arbitrary value for caster wheel mass -->
-        <xacro:property name="caster_wheel_radius" value="0.015" />
         <xacro:property name="z_offset" value="-${base_height/2}" />
         <!-- Space btw top of beam and the each joint -->
+        <xacro:macro name="wheel" params="name x y">
+            <joint name="${name}_joint" type="continuous">
+                <parent link="base_link"/>
+                <child link="${name}"/>
+                <origin xyz="${x} ${y} ${z_offset}" rpy="0 0 0"/>
+                <axis xyz="0 1 0"/>
+                <dynamics damping="0.2"/>
+            </joint>
+            <link name="${name}">
+                <collision>
+                    <origin xyz="0 0 0" rpy="${PI/2} 0 0"/>
+                    <geometry>
+                        <cylinder length="${wheel_len}" radius="${wheel_radius}"/>
+                    </geometry>
+                </collision>
+                <visual>
+                    <origin xyz="0 0 0" rpy="${PI/2} 0 0"/>
+                    <geometry>
+                        <cylinder length="${wheel_len}" radius="${wheel_radius}"/>
+                    </geometry>
+                    <material name="black"/>
+                </visual>
+                <inertial>
+                    <origin xyz="0 0 0" rpy="${PI/2} 0 0"/>
+                    <mass value="${wheel_mass}"/>
+                    <inertia ixx="${wheel_mass / 12.0 * (3*wheel_radius + wheel_len*wheel_len)}" ixy="0.0" ixz="0.0" iyy="${wheel_mass / 12.0 * wheel_radius*wheel_radius}" iyz="0.0" izz="${wheel_mass / 12.0 * wheel_radius*wheel_radius}"/>
+                </inertial>
+            </link>
+        </xacro:macro>
         <!-- Base Link -->
         <link name="base_link">
@@ -39,59 +65,10 @@
             </inertial>
         </link>
-        <joint name="left_wheel_joint" type="continuous">
-            <parent link="base_link"/>
-            <child link="left_wheel"/>
-            <origin xyz="0 -${base_width/2} ${z_offset}" rpy="0 0 0"/>
-            <axis xyz="0 1 0"/>
-            <dynamics damping="0.2"/>
-        </joint>
-        <!-- left front wheel Link -->
-        <link name="left_wheel">
-            <origin xyz="0 0 0" rpy="${PI/2} 0 0"/>
-            <geometry>
-                <cylinder length="${wheel_len}" radius="${wheel_radius}"/>
-            </geometry>
-        </collision>
-        <visual>
-            <origin xyz="0 0 0" rpy="${PI/2} 0 0"/>
-            <geometry>
-                <cylinder length="${wheel_len}" radius="${wheel_radius}"/>
-            </geometry>
-            <material name="black"/>
-        </visual>
-        <inertial>
-            <origin xyz="0 0 0" rpy="${PI/2} 0 0"/>
-            <mass value="${wheel_mass}"/>
-            <inertia ixx="${wheel_mass / 12.0 * (3*wheel_radius + wheel_len*wheel_len)}" ixy="0.0" ixz="0.0" iyy="${wheel_mass / 12.0 * wheel_radius*wheel_radius}" iyz="0.0" izz="${wheel_mass / 12.0 * wheel_radius*wheel_radius}"/>
-        </inertial>
-    </link>
-    <joint name="right_wheel_joint" type="continuous">
-        <parent link="base_link"/>
-        <child link="right_wheel"/>
-        <origin xyz="0 ${base_width/2} ${z_offset}" rpy="0 0 0"/>
-        <axis xyz="0 1 0"/>
-        <dynamics damping="0.2"/>
-    </joint>
-    <!-- right wheel Link -->
-    <link name="right_wheel">
-        <collision>
-            <origin xyz="0 0 0" rpy="${PI/2} 0 0"/>
-            <geometry>
-                <cylinder length="${wheel_len}" radius="${wheel_radius}"/>
-            </geometry>
-        </collision>
-        <visual>
-            <origin xyz="0 0 0" rpy="${PI/2} 0 0"/>
-            <geometry>
-                <cylinder length="${wheel_len}" radius="${wheel_radius}"/>
-            </geometry>
-            <material name="black"/>
-        </visual>
-        <inertial>
-            <origin xyz="0 0 0" rpy="${PI/2} 0 0"/>
-            <mass value="${wheel_mass}"/>
-            <inertia ixx="${wheel_mass / 12.0 * (3*wheel_radius + wheel_len*wheel_len)}" ixy="0.0" ixz="0.0" iyy="${wheel_mass / 12.0 * wheel_radius*wheel_radius}" iyz="0.0" izz="${wheel_mass / 12.0 * wheel_radius*wheel_radius}"/>
-        </inertial>
-    </link>
-</xacro:macro>
+        <xacro:wheel name="left_front" x="${base_width/2}" y="-${base_width/2}" />
+        <xacro:wheel name="left_mid" x="0" y="-${base_width/2}" />
+        <xacro:wheel name="left_back" x="-${base_width/2}" y="-${base_width/2}" />
+        <xacro:wheel name="right_front" x="${base_width/2}" y="${base_width/2}" />
+        <xacro:wheel name="right_mid" x="0" y="${base_width/2}" />
+        <xacro:wheel name="right_back" x="-${base_width/2}" y="${base_width/2}" />
+    </xacro:macro>
 </robot>
