Commit message: Arm with controller

File: src/cmr_description/cmr_arm_description/urdf/arm_description.urdf.xacro (robot description, xacro)
@@ -7,22 +7,23 @@
 Note that most links have origins equal to half their lengths.
  -->
-<robot name="arm_description"
-  xmlns:xacro="http://ros.org/wiki/xacro">
-  <xacro:include filename="arm_macros.urdf.xacro" />
-  <xacro:linkage name="base" origin_xyz="0 0 0" origin_rpy="0 0 0" length="0" radius=".0001" color="0 1 0 1" mass="1000"/>
-  <xacro:linkage name="base_rotate" origin_xyz="0 0 0" origin_rpy="0 0 0" length="0.05" radius="0.2" color="1 0 0 1" mass="1" mesh="base_rotate" vOrigin_xyz="0 0 0" vOrigin_rpy="-1.57 3.14 0"/>
-  <xacro:joint_rev name="base_rotate" origin_xyz="0 0 0" parent="base" child="base_rotate" axis="0 0 1" lower_limit="-1.57" upper_limit="1.57"/>
-  <xacro:linkage name="shoulder" origin_xyz="0 0 0.17215" origin_rpy="0 0 0" length="0.3443" radius="0.04" color="1 0 0 1" mass=".65" mesh="shoulder" vOrigin_xyz=".027 0.085 -0.065" vOrigin_rpy="2.35 -0.1 0.05"/>
-  <xacro:joint_rev name="shoulder" origin_xyz="0 0 0.098" parent="base_rotate" child="shoulder" axis="1 0 0" lower_limit="-1.57" upper_limit="1.57"/>
-  <xacro:linkage name="elbow" origin_xyz="0.049 0 0" origin_rpy="0 1.57075 0" length="0.098" radius="0.02" color="0 0 1 1" mass=".10" mesh="shoulder_elbow_joint" vOrigin_xyz="0.002 .35 -.235" vOrigin_rpy="3.14 -.1 0"/>
-  <xacro:joint_rev name="elbow" origin_xyz="0 0 0.3443" parent="shoulder" child="elbow" axis="1 0 0" lower_limit="-2.35" upper_limit="2.35"/>
-  <xacro:linkage name="second_rotate" origin_xyz="0 0 0.2298" origin_rpy="0 0 0" length="0.4596" radius="0.02" color="0 0.5 0.5 1" mass=".65" mesh="elbow" vOrigin_xyz="-0.083 0.35 -0.24" vOrigin_rpy="3.14 -0.15 0"/>
-  <xacro:joint_rev name="second_rotate" origin_xyz="0.098 0 0" parent="elbow" child="second_rotate" axis="0 0 1" lower_limit="-3.14" upper_limit="3.14"/>
-  <xacro:linkage name="third_tilt" origin_xyz="0 0 0.0674" origin_rpy="0 0 0" length="0.1348" radius="0.02" color=".4 .3 .3 1" mass=".30" mesh="second_tilt" vOrigin_xyz="-.164 0.72 -.255" vOrigin_rpy="-2.355 -0.1 0"/>
-  <xacro:joint_rev name="third_tilt" origin_xyz="0 0 0.4596" parent="second_rotate" child="third_tilt" axis="1 0 0" lower_limit="-1.57" upper_limit="1.57"/>
-  <xacro:linkage name="third_rotate" origin_xyz="0 0 0.0726" origin_rpy="0 0 0" length="0.1452" radius="0.02" color="1 1 1 1" mass=".30" mesh="end_effector" vOrigin_xyz="0 0 0" vOrigin_rpy="0 0 0"/>
-  <xacro:joint_continuous name="third_rotate" origin_xyz="0 0 0.1348" parent="third_tilt" child="third_rotate" axis="0 0 1"/>
-  <xacro:linkage name="end_effector" origin_xyz="0 0 0.012" origin_rpy="0 0 0" length="0.025" radius="0.025" color="0 0 0 1" mass=".30"/>
-  <!-- The Last Joint is effectively fixed, and exists at the tip of the end effector -->
-  <xacro:joint_rev name="end_effector" origin_xyz="0 0 0.1702" origin_rpy="-1 0 0" parent="third_rotate" child="end_effector" axis="0 0 1" lower_limit="0" upper_limit="0" />
+<robot xmlns:xacro="http://www.ros.org/wiki/xacro">
+  <xacro:macro name="arm">
+    <xacro:include filename="arm_macros.urdf.xacro" />
+    <xacro:linkage name="base" origin_xyz="0 0 0" origin_rpy="0 0 0" length="0" radius=".0001" color="0 1 0 1" mass="1000"/>
+    <xacro:linkage name="base_rotate" origin_xyz="0 0 0" origin_rpy="0 0 0" length="0.05" radius="0.2" color="1 0 0 1" mass="1" mesh="base_rotate" vOrigin_xyz="0 0 0" vOrigin_rpy="-1.57 3.14 0"/>
+    <xacro:joint_rev name="base_rotate" origin_xyz="0 0 0" parent="base" child="base_rotate" axis="0 0 1" lower_limit="-1.57" upper_limit="1.57"/>
+    <xacro:linkage name="shoulder" origin_xyz="0 0 0.17215" origin_rpy="0 0 0" length="0.3443" radius="0.04" color="1 0 0 1" mass=".65" mesh="shoulder" vOrigin_xyz=".027 0.085 -0.065" vOrigin_rpy="2.35 -0.1 0.05"/>
+    <xacro:joint_rev name="shoulder" origin_xyz="0 0 0.098" parent="base_rotate" child="shoulder" axis="1 0 0" lower_limit="-1.57" upper_limit="1.57"/>
+    <xacro:linkage name="elbow" origin_xyz="0.049 0 0" origin_rpy="0 1.57075 0" length="0.098" radius="0.02" color="0 0 1 1" mass=".10" mesh="shoulder_elbow_joint" vOrigin_xyz="0.002 .35 -.235" vOrigin_rpy="3.14 -.1 0"/>
+    <xacro:joint_rev name="elbow" origin_xyz="0 0 0.3443" parent="shoulder" child="elbow" axis="1 0 0" lower_limit="-2.35" upper_limit="2.35"/>
+    <xacro:linkage name="second_rotate" origin_xyz="0 0 0.2298" origin_rpy="0 0 0" length="0.4596" radius="0.02" color="0 0.5 0.5 1" mass=".65" mesh="elbow" vOrigin_xyz="-0.083 0.35 -0.24" vOrigin_rpy="3.14 -0.15 0"/>
+    <xacro:joint_rev name="second_rotate" origin_xyz="0.098 0 0" parent="elbow" child="second_rotate" axis="0 0 1" lower_limit="-3.14" upper_limit="3.14"/>
+    <xacro:linkage name="third_tilt" origin_xyz="0 0 0.0674" origin_rpy="0 0 0" length="0.1348" radius="0.02" color=".4 .3 .3 1" mass=".30" mesh="second_tilt" vOrigin_xyz="-.164 0.72 -.255" vOrigin_rpy="-2.355 -0.1 0"/>
+    <xacro:joint_rev name="third_tilt" origin_xyz="0 0 0.4596" parent="second_rotate" child="third_tilt" axis="1 0 0" lower_limit="-1.57" upper_limit="1.57"/>
+    <xacro:linkage name="third_rotate" origin_xyz="0 0 0.0726" origin_rpy="0 0 0" length="0.1452" radius="0.02" color="1 1 1 1" mass=".30" mesh="end_effector" vOrigin_xyz="0 0 0" vOrigin_rpy="0 0 0"/>
+    <xacro:joint_continuous name="third_rotate" origin_xyz="0 0 0.1348" parent="third_tilt" child="third_rotate" axis="0 0 1"/>
+    <xacro:linkage name="end_effector" origin_xyz="0 0 0.012" origin_rpy="0 0 0" length="0.025" radius="0.025" color="0 0 0 1" mass=".30"/>
+    <!-- The Last Joint is effectively fixed, and exists at the tip of the end effector -->
+    <xacro:joint_rev name="end_effector" origin_xyz="0 0 0.1702" origin_rpy="-1 0 0" parent="third_rotate" child="end_effector" axis="0 0 1" lower_limit="0" upper_limit="0" />
+  </xacro:macro>
 </robot>
