Commit message: Support mocking

File: src/cmr_description/cmr_arm_description/ros2_control/arm.ros2_control.xacro (robot description, xacro)
@@ -1,8 +1,13 @@
 <?xml version="1.0"?>
 <robot xmlns:xacro="http://www.ros.org/wiki/xacro">
-    <xacro:macro name="arm_ros2_control" params="name">
+    <xacro:macro name="arm_ros2_control" params="name mock">
         <ros2_control name="${name}" type="system">
             <hardware>
-                <plugin>cmr_control/MockArmSystemHardware</plugin>
+                <xacro:if value="${mock}">
+                    <plugin>cmr_control/MockArmSystemHardware</plugin>
+                </xacro:if>
+                <xacro:unless value="${mock}">
+                    <plugin>cmr_control/ArmSystemHardware</plugin>
+                </xacro:unless>
             </hardware>
             <joint name="base_rotate">

File: src/cmr_description/cmr_arm_description/urdf/arm.urdf.xacro (robot description, xacro)
@@ -2,9 +2,8 @@
 <robot xmlns:xacro="http://www.ros.org/wiki/xacro" name="drives">
     <xacro:arg name="use_gazebo" default="false" />
-    <xacro:arg name="use_fake_hardware" default="true" />
-    <xacro:arg name="fake_sensor_commands" default="false" />
+    <xacro:arg name="mock" default="true" />
     <xacro:include filename="$(find cmr_arm_description)/urdf/arm_description.urdf.xacro" />
     <xacro:include filename="$(find cmr_arm_description)/ros2_control/arm.ros2_control.xacro" />
     <xacro:arm />
-    <xacro:arm_ros2_control name="arm"/>
+    <xacro:arm_ros2_control name="arm" mock="$(arg mock)"/>
 </robot>
