Commit message: Astrotech Motor Hardware Interface (#40)
* Astrotech motor control

* should be done now

* Astro motor spinny thingy ad-hoc test setup

* AstroMotor small cleanup changes

* Astro motor control and tests

Co-authored-by: Arden <apl88@cornell.edu>

File: src/cmr_description/cmr_drives_description/urdf/drives.urdf.xacro (robot description, xacro)
@@ -8,6 +8,8 @@
     <xacro:include filename="$(find cmr_drives_description)/ros2_control/drives.ros2_control.xacro" />
     <xacro:include filename="$(find cmr_drives_description)/ros2_control/sensor.ros2_control.xacro" />
+    <xacro:include filename="$(find cmr_drives_description)/ros2_control/astro_motor.ros2_control.xacro" />
     <xacro:drives />
     <xacro:drives_ros2_control name="drives"/>
     <xacro:astro_sensor name="test_astro_sensor" prefix="test_"/>
+    <xacro:astro_motor_ros2_control name="test_astro_motor" joint="test_astro_joint" />
 </robot>

File: src/cmr_description/cmr_drives_description/urdf/drives_description.urdf.xacro (robot description, xacro)
@@ -25,4 +25,8 @@
         <xacro:property name="imu_height" value="${base_height / 2.0}" />
         <xacro:property name="imu_length" value="${base_length}" />
+        <xacro:property name="astro_length" value="0.1" />
+        <xacro:property name="astro_width" value="0.3" />
+        <xacro:property name="astro_height" value="0.03" />
+        <xacro:property name="astro_mass" value="${base_mass / 3}" />
         <!-- Space btw top of beam and the each joint -->
         <xacro:macro name="wheel" params="name x y">
@@ -202,4 +206,34 @@
         <xacro:wheel name="right_mid" x="0" y="${base_length/2 + wheel_len}" />
         <xacro:wheel name="right_back" x="-${base_width/2}" y="${base_length/2 + wheel_len}" />
+        <!-- Test astro link -->
+        <link name="test_astro">
+            <collision>
+                <origin xyz="0 0 0" rpy="0 0 0"/>
+                <geometry>
+                    <box size="${astro_width} ${astro_length} ${astro_height}"/>
+                </geometry>
+            </collision>
+            <visual>
+                <origin xyz="0 0 0" rpy="0 0 0"/>
+                <geometry>
+                    <box size="${astro_width} ${astro_length} ${astro_height}"/>
+                </geometry>
+                <material name="blue"/>
+            </visual>
+            <inertial>
+                <origin xyz="0 0 0" rpy="0 0 0"/>
+                <mass value="${astro_mass}"/>
+                <inertia ixx="${astro_mass / 12.0 * (astro_length*astro_length + astro_height*astro_height)}" ixy="0.0" ixz="0.0"
+                         iyy="${astro_mass / 12.0 * astro_width*astro_width}" iyz="0.0"
+                         izz="${astro_mass / 12.0 * (astro_width*astro_width + astro_length*astro_length)}"/>
+            </inertial>
+        </link>
+        <joint name="test_astro_joint" type="continuous">
+            <parent link="base_link"/>
+            <child link="test_astro"/>
+            <origin xyz="${-astro_width / 2.0} 0 ${base_height * 2 + lidar_height}" rpy="0 0 0"/>
+            <axis xyz="0 0 1"/>
+            <dynamics damping="0.2"/>
+        </joint>
     </xacro:macro>
     <gazebo reference="imu_link">
