Commit message: Add joint state publisher

File: src/cmr_description/cmr_drives_description/urdf/drives_description.urdf.xacro (robot description, xacro)
@@ -1,5 +1,5 @@
 <?xml version="1.0"?>
 <robot xmlns:xacro="http://www.ros.org/wiki/xacro">
-    <xacro:macro name="drives" params="">
+    <xacro:macro name="drives">
         <!-- Constants for robot dimensions -->
         <xacro:property name="PI" value="3.1415926535897931"/>
@@ -46,105 +46,52 @@
             <dynamics damping="0.2"/>
         </joint>
-        <!-- left wheel Link -->
+        <!-- left front wheel Link -->
         <link name="left_wheel">
-            <collision>
-                <origin xyz="0 0 0" rpy="${PI/2} 0 0"/>
-                <geometry>
-                    <cylinder length="${wheel_len}" radius="${wheel_radius}"/>
-                </geometry>
-            </collision>
-            <visual>
-                <origin xyz="0 0 0" rpy="${PI/2} 0 0"/>
-                <geometry>
-                    <cylinder length="${wheel_len}" radius="${wheel_radius}"/>
-                </geometry>
-                <material name="black"/>
-            </visual>
-            <inertial>
-                <origin xyz="0 0 0" rpy="${PI/2} 0 0"/>
-                <mass value="${wheel_mass}"/>
-                <inertia ixx="${wheel_mass / 12.0 * (3*wheel_radius + wheel_len*wheel_len)}" ixy="0.0" ixz="0.0" iyy="${wheel_mass / 12.0 * wheel_radius*wheel_radius}" iyz="0.0" izz="${wheel_mass / 12.0 * wheel_radius*wheel_radius}"/>
-            </inertial>
-        </link>
-        <joint name="right_wheel_joint" type="continuous">
-            <parent link="base_link"/>
-            <child link="right_wheel"/>
-            <origin xyz="0 ${base_width/2} ${z_offset}" rpy="0 0 0"/>
-            <axis xyz="0 1 0"/>
-            <dynamics damping="0.2"/>
-        </joint>
-        <!-- right wheel Link -->
-        <link name="right_wheel">
-            <collision>
-                <origin xyz="0 0 0" rpy="${PI/2} 0 0"/>
-                <geometry>
-                    <cylinder length="${wheel_len}" radius="${wheel_radius}"/>
-                </geometry>
-            </collision>
-            <visual>
-                <origin xyz="0 0 0" rpy="${PI/2} 0 0"/>
-                <geometry>
-                    <cylinder length="${wheel_len}" radius="${wheel_radius}"/>
-                </geometry>
-                <material name="black"/>
-            </visual>
-            <inertial>
-                <origin xyz="0 0 0" rpy="${PI/2} 0 0"/>
-                <mass value="${wheel_mass}"/>
-                <inertia ixx="${wheel_mass / 12.0 * (3*wheel_radius + wheel_len*wheel_len)}" ixy="0.0" ixz="0.0" iyy="${wheel_mass / 12.0 * wheel_radius*wheel_radius}" iyz="0.0" izz="${wheel_mass / 12.0 * wheel_radius*wheel_radius}"/>
-            </inertial>
-        </link>
-        <joint name="caster_frontal_wheel_joint" type="fixed">
-            <parent link="base_link"/>
-            <child link="caster_frontal_wheel"/>
-            <origin xyz="${base_width/2 - caster_wheel_radius} 0 ${z_offset}" rpy="0 0 0"/>
-        </joint>
-        <!-- caster frontal wheel Link -->
-        <link name="caster_frontal_wheel">
-            <collision>
-                <origin xyz="0 0 0" rpy="0 0 0"/>
-                <geometry>
-                    <sphere radius="${caster_wheel_radius}"/>
-                </geometry>
-            </collision>
-            <visual>
-                <origin xyz="0 0 0" rpy="0 0 0"/>
-                <geometry>
-                    <sphere radius="${caster_wheel_radius}"/>
-                </geometry>
-                <material name="white"/>
-            </visual>
-            <inertial>
-                <origin xyz="0 0 0" rpy="0 0 0"/>
-                <mass value="${caster_wheel_mass}"/>
-                <inertia ixx="${caster_wheel_mass * 0.4 * (caster_wheel_radius * caster_wheel_radius)}" ixy="0.0" ixz="0.0" iyy="${caster_wheel_mass * 0.4 * (caster_wheel_radius * caster_wheel_radius)}" iyz="0.0" izz="${caster_wheel_mass * 0.4 * (caster_wheel_radius * caster_wheel_radius)}"/>
-            </inertial>
-        </link>
-        <joint name="caster_rear_wheel_joint" type="fixed">
-            <parent link="base_link"/>
-            <child link="caster_rear_wheel"/>
-            <origin xyz="${-base_width/2 + caster_wheel_radius} 0 ${z_offset}" rpy="0 0 0"/>
-        </joint>
-        <!-- caster rear wheel Link -->
-        <link name="caster_rear_wheel">
-            <collision>
-                <origin xyz="0 0 0" rpy="0 0 0"/>
-                <geometry>
-                    <sphere radius="${caster_wheel_radius}"/>
-                </geometry>
-            </collision>
-            <visual>
-                <origin xyz="0 0 0" rpy="0 0 0"/>
-                <geometry>
-                    <sphere radius="${caster_wheel_radius}"/>
-                </geometry>
-                <material name="white"/>
-            </visual>
-            <inertial>
-                <origin xyz="0 0 0" rpy="0 0 0"/>
-                <mass value="${caster_wheel_mass}"/>
-                <inertia ixx="${caster_wheel_mass * 0.4 * (caster_wheel_radius * caster_wheel_radius)}" ixy="0.0" ixz="0.0" iyy="${caster_wheel_mass * 0.4 * (caster_wheel_radius * caster_wheel_radius)}" iyz="0.0" izz="${caster_wheel_mass * 0.4 * (caster_wheel_radius * caster_wheel_radius)}"/>
-            </inertial>
-        </link>
-    </xacro:macro>
+            <origin xyz="0 0 0" rpy="${PI/2} 0 0"/>
+            <geometry>
+                <cylinder length="${wheel_len}" radius="${wheel_radius}"/>
+            </geometry>
+        </collision>
+        <visual>
+            <origin xyz="0 0 0" rpy="${PI/2} 0 0"/>
+            <geometry>
+                <cylinder length="${wheel_len}" radius="${wheel_radius}"/>
+            </geometry>
+            <material name="black"/>
+        </visual>
+        <inertial>
+            <origin xyz="0 0 0" rpy="${PI/2} 0 0"/>
+            <mass value="${wheel_mass}"/>
+            <inertia ixx="${wheel_mass / 12.0 * (3*wheel_radius + wheel_len*wheel_len)}" ixy="0.0" ixz="0.0" iyy="${wheel_mass / 12.0 * wheel_radius*wheel_radius}" iyz="0.0" izz="${wheel_mass / 12.0 * wheel_radius*wheel_radius}"/>
+        </inertial>
+    </link>
+    <joint name="right_wheel_joint" type="continuous">
+        <parent link="base_link"/>
+        <child link="right_wheel"/>
+        <origin xyz="0 ${base_width/2} ${z_offset}" rpy="0 0 0"/>
+        <axis xyz="0 1 0"/>
+        <dynamics damping="0.2"/>
+    </joint>
+    <!-- right wheel Link -->
+    <link name="right_wheel">
+        <collision>
+            <origin xyz="0 0 0" rpy="${PI/2} 0 0"/>
+            <geometry>
+                <cylinder length="${wheel_len}" radius="${wheel_radius}"/>
+            </geometry>
+        </collision>
+        <visual>
+            <origin xyz="0 0 0" rpy="${PI/2} 0 0"/>
+            <geometry>
+                <cylinder length="${wheel_len}" radius="${wheel_radius}"/>
+            </geometry>
+            <material name="black"/>
+        </visual>
+        <inertial>
+            <origin xyz="0 0 0" rpy="${PI/2} 0 0"/>
+            <mass value="${wheel_mass}"/>
+            <inertia ixx="${wheel_mass / 12.0 * (3*wheel_radius + wheel_len*wheel_len)}" ixy="0.0" ixz="0.0" iyy="${wheel_mass / 12.0 * wheel_radius*wheel_radius}" iyz="0.0" izz="${wheel_mass / 12.0 * wheel_radius*wheel_radius}"/>
+        </inertial>
+    </link>
+</xacro:macro>
 </robot>
