Commit message: Autonomy Gazebo Simulation (#31)
* current urdf and launch files

* Added sensors to urdf and added world file

* gazebo works, error in reading urdf properly

* gazebo is able to run

* Modified scripts

* Diff drives, camera, lidar

* SLAM

* Remove old nav WIP

* use modern cmr_install and remove unused config

* Remove unused empty world

Co-authored-by: ap736 <ap736@cornell.edu>
Co-authored-by: Avocado <cmravocado@gmail.com>

File: src/cmr_description/cmr_drives_description/urdf/drives_description.urdf.xacro (robot description, xacro)
@@ -4,14 +4,25 @@
         <!-- Constants for robot dimensions -->
         <xacro:property name="PI" value="3.1415926535897931"/>
-        <xacro:property name="base_mass" value="0.3" />
+        <xacro:property name="base_mass" value="20" />
+        <xacro:property name="lidar_mass" value="8" />
+        <xacro:property name="camera_mass" value="8" />
+        <xacro:property name="imu_mass" value="12" />
         <!-- arbitrary value for base mass -->
-        <xacro:property name="base_width" value="0.1" />
-        <xacro:property name="base_length" value="0.1" />
-        <xacro:property name="base_height" value="0.05" />
-        <xacro:property name="wheel_mass" value="0.3" />
+        <xacro:property name="base_width" value="1" />
+        <xacro:property name="base_length" value="0.5" />
+        <xacro:property name="base_height" value="0.1" />
+        <xacro:property name="wheel_mass" value="5" />
         <!-- arbitrary value for wheel mass -->
-        <xacro:property name="wheel_len" value="0.020" />
-        <xacro:property name="wheel_radius" value="0.015" />
+        <xacro:property name="wheel_len" value="0.1" />
+        <xacro:property name="wheel_radius" value="0.1" />
         <xacro:property name="z_offset" value="-${base_height/2}" />
+        <xacro:property name="lidar_radius" value="0.1" />
+        <xacro:property name="lidar_height" value="${base_height/2}" />
+        <xacro:property name="cam_width" value="${base_length / 5.0}" />
+        <xacro:property name="cam_height" value="${base_height / 10.0}" />
+        <xacro:property name="cam_length" value="${base_length / 10.0}" />
+        <xacro:property name="imu_width" value="${base_width}" />
+        <xacro:property name="imu_height" value="${base_height / 2.0}" />
+        <xacro:property name="imu_length" value="${base_length}" />
         <!-- Space btw top of beam and the each joint -->
         <xacro:macro name="wheel" params="name x y">
@@ -43,4 +54,34 @@
                 </inertial>
             </link>
+            <gazebo reference="${name}">
+                <!-- <mu>1000</mu>
+                <mu1>1000</mu1>
+                <mu2>1000</mu2>
+                <kp>1000000.0</kp>
+                <kd>100.0</kd>
+                <fdir1 value="1 0 0"/>
+                <max_vel>1.0</max_vel>
+                <min_depth>0.00</min_depth> -->
+                <surface>
+                  <friction>
+                    <ode>
+                      <mu>1.5</mu>
+                      <mu2>1.5</mu2>
+                      <slip1>0</slip1>
+                      <slip2>0</slip2>
+                    </ode>
+                  </friction>
+                   <contact>
+                    <ode>
+                      <soft_cfm>0</soft_cfm>
+                      <soft_erp>0.2</soft_erp>
+                      <kp>1e+13</kp>
+                      <kd>1</kd>
+                      <max_vel>1</max_vel>
+                      <min_depth>0.01</min_depth>
+                    </ode>
+                  </contact>
+                </surface>
+              </gazebo>
         </xacro:macro>
         <!-- Base Link -->
@@ -65,10 +106,273 @@
             </inertial>
         </link>
-        <xacro:wheel name="left_front" x="${base_width/2}" y="-${base_width/2}" />
-        <xacro:wheel name="left_mid" x="0" y="-${base_width/2}" />
-        <xacro:wheel name="left_back" x="-${base_width/2}" y="-${base_width/2}" />
-        <xacro:wheel name="right_front" x="${base_width/2}" y="${base_width/2}" />
-        <xacro:wheel name="right_mid" x="0" y="${base_width/2}" />
-        <xacro:wheel name="right_back" x="-${base_width/2}" y="${base_width/2}" />
+        <!-- Lidar Link -->
+        <link name="lidar_link">
+            <inertial>
+                <origin xyz="0 0 0" rpy="0 0 0"/>
+                <mass value="${lidar_mass}"/>
+                <inertia ixx="${lidar_mass / 12.0 * (3.0 * lidar_radius * lidar_radius + lidar_height * lidar_height)}"
+                         ixy="0"
+                         ixz="0"
+                         iyy="${lidar_mass / 12.0 * (3.0 * lidar_radius * lidar_radius + lidar_height * lidar_height)}"
+                         iyz="0"
+                         izz="${0.5 * lidar_mass * lidar_radius * lidar_radius}" />
+            </inertial>
+            <collision>
+                <origin xyz="0 0 0" rpy="0 0 0"/>
+                <geometry>
+                    <cylinder radius="${lidar_radius}" length="${lidar_height}"/>
+                </geometry>
+            </collision>
+            <visual>
+                <origin xyz="0 0 0" rpy="0 0 0"/>
+                <geometry>
+                    <cylinder radius="${lidar_radius}" length="${lidar_height}"/>
+                </geometry>
+            </visual>
+        </link>
+        <joint name="lidar_joint" type="fixed">
+            <parent link="base_link"/>
+            <child link="lidar_link"/>
+            <origin xyz="0 0 ${base_height*2}" rpy="0 0 0"/>
+        </joint>
+        <!-- IMU Link -->
+        <link name="imu_link">
+            <visual>
+                <geometry>
+                    <box size="${imu_width} ${imu_length} ${imu_height}"/>
+                </geometry>
+            </visual>
+            <collision>
+                <geometry>
+                    <box size="${imu_width} ${imu_length} ${imu_height}"/>
+                </geometry>
+            </collision>
+            <!-- <xacro:box_inertia m="0.1" w="0.1" d="0.1" h="0.1"/> -->
+            <inertial>
+                <origin xyz="0 0 0" rpy="0 0 0"/>
+                <mass value="${imu_mass}"/>
+                <inertia ixx="${imu_mass / 12.0 * (imu_height * imu_height + imu_length * imu_length)}"
+                         ixy="0"
+                         ixz="0"
+                         iyy="${imu_mass / 12.0 * (imu_height * imu_height + imu_width * imu_width)}"
+                         iyz="0"
+                         izz="${imu_mass / 12.0 * (imu_width * imu_width + imu_length * imu_length)}" />
+            </inertial>
+        </link>
+        <joint name="imu_joint" type="fixed">
+            <parent link="base_link"/>
+            <child link="imu_link"/>
+            <origin xyz="0 0 ${base_height * 1.25}"/>
+        </joint>
+        <!-- Camera Link -->
+        <link name="camera_link">
+            <visual>
+                <origin xyz="0 0 0" rpy="0 0 0"/>
+                <geometry>
+                    <box size="${cam_width} ${cam_length} ${cam_height}"/>
+                </geometry>
+            </visual>
+            <collision>
+                <origin xyz="0 0 0" rpy="0 0 0"/>
+                <geometry>
+                    <box size="${cam_width} ${cam_length} ${cam_height}"/>
+                </geometry>
+            </collision>
+            <inertial>
+                <origin xyz="0 0 0" rpy="0 0 0"/>
+                <mass value="${camera_mass}"/>
+                <inertia ixx="${camera_mass / 12.0 * (cam_height * cam_height + cam_length * cam_length)}"
+                         ixy="0"
+                         ixz="0"
+                         iyy="${camera_mass / 12.0 * (cam_height * cam_height + cam_width * cam_width)}"
+                         iyz="0"
+                         izz="${camera_mass / 12.0 * (cam_width * cam_width + cam_length * cam_length)}" />
+            </inertial>
+        </link>
+        <joint name="camera_joint" type="fixed">
+            <parent link="base_link"/>
+            <child link="camera_link"/>
+            <origin xyz="${base_width / 2} 0 ${base_height}" rpy="0 0 0"/>
+        </joint>
+        <!-- Wheels -->
+        <xacro:wheel name="left_front" x="${base_width/2}" y="-${base_length/2 + wheel_len}" />
+        <xacro:wheel name="left_mid" x="0" y="-${base_length/2 + wheel_len}" />
+        <xacro:wheel name="left_back" x="-${base_width/2}" y="-${base_length/2 + wheel_len}" />
+        <xacro:wheel name="right_front" x="${base_width/2}" y="${base_length/2 + wheel_len}" />
+        <xacro:wheel name="right_mid" x="0" y="${base_length/2 + wheel_len}" />
+        <xacro:wheel name="right_back" x="-${base_width/2}" y="${base_length/2 + wheel_len}" />
     </xacro:macro>
+    <gazebo reference="imu_link">
+        <sensor name="imu_sensor" type="imu">
+            <plugin filename="libgazebo_ros_imu_sensor.so" name="imu_plugin">
+                <ros>
+                    <namespace>/demo</namespace>
+                    <remapping>~/out:=imu</remapping>
+                </ros>
+                <initial_orientation_as_reference>false</initial_orientation_as_reference>
+            </plugin>
+            <always_on>true</always_on>
+            <update_rate>100</update_rate>
+            <visualize>true</visualize>
+            <imu>
+                <angular_velocity>
+                    <x>
+                        <noise type="gaussian">
+                            <mean>0.0</mean>
+                            <stddev>2e-4</stddev>
+                            <bias_mean>0.0000075</bias_mean>
+                            <bias_stddev>0.0000008</bias_stddev>
+                        </noise>
+                    </x>
+                    <y>
+                        <noise type="gaussian">
+                            <mean>0.0</mean>
+                            <stddev>2e-4</stddev>
+                            <bias_mean>0.0000075</bias_mean>
+                            <bias_stddev>0.0000008</bias_stddev>
+                        </noise>
+                    </y>
+                    <z>
+                        <noise type="gaussian">
+                            <mean>0.0</mean>
+                            <stddev>2e-4</stddev>
+                            <bias_mean>0.0000075</bias_mean>
+                            <bias_stddev>0.0000008</bias_stddev>
+                        </noise>
+                    </z>
+                </angular_velocity>
+                <linear_acceleration>
+                    <x>
+                        <noise type="gaussian">
+                            <mean>0.0</mean>
+                            <stddev>1.7e-2</stddev>
+                            <bias_mean>0.1</bias_mean>
+                            <bias_stddev>0.001</bias_stddev>
+                        </noise>
+                    </x>
+                    <y>
+                        <noise type="gaussian">
+                            <mean>0.0</mean>
+                            <stddev>1.7e-2</stddev>
+                            <bias_mean>0.1</bias_mean>
+                            <bias_stddev>0.001</bias_stddev>
+                        </noise>
+                    </y>
+                    <z>
+                        <noise type="gaussian">
+                            <mean>0.0</mean>
+                            <stddev>1.7e-2</stddev>
+                            <bias_mean>0.1</bias_mean>
+                            <bias_stddev>0.001</bias_stddev>
+                        </noise>
+                    </z>
+                </linear_acceleration>
+            </imu>
+        </sensor>
+    </gazebo>
+    <gazebo>
+        <plugin name='diff_drive' filename='libgazebo_ros_diff_drive.so'>
+            <ros>
+                <namespace>/</namespace>
+            </ros>
+            <!-- wheels -->
+            <num_wheel_pairs>3</num_wheel_pairs>
+            <left_joint>left_front_joint</left_joint>
+            <left_joint>left_mid_joint</left_joint>
+            <left_joint>left_back_joint</left_joint>
+            <right_joint>right_front_joint</right_joint>
+            <right_joint>right_mid_joint</right_joint>
+            <right_joint>right_back_joint</right_joint>
+            <!-- kinematics -->
+            <wheel_separation>0.5</wheel_separation>
+            <wheel_diameter>0.2</wheel_diameter>
+            <!-- limits -->
+            <max_wheel_torque>500</max_wheel_torque>
+            <max_wheel_acceleration>10.0</max_wheel_acceleration>
+            <!-- output -->
+            <odom_publish_frequency>1</odom_publish_frequency>
+            <publish_odom>true</publish_odom>
+            <publish_odom_tf>true</publish_odom_tf>
+            <publish_wheel_tf>true</publish_wheel_tf>
+            <odom_topic>/odom</odom_topic>
+            <topic>/cmd_vel</topic>
+            <source_frame>map</source_frame>
+            <odometry_frame>odom</odometry_frame>
+            <robot_base_frame>base_link</robot_base_frame>
+        </plugin>
+    </gazebo>
+    <gazebo reference="lidar_link">
+        <sensor name="lidar" type="ray">
+            <always_on>true</always_on>
+            <visualize>true</visualize>
+            <update_rate>5</update_rate>
+            <ray>
+                <scan>
+                    <horizontal>
+                        <samples>360</samples>
+                        <resolution>1.000000</resolution>
+                        <min_angle>0.000000</min_angle>
+                        <max_angle>6.280000</max_angle>
+                    </horizontal>
+                </scan>
+                <range>
+                    <min>0.120000</min>
+                    <max>3.5</max>
+                    <resolution>0.015000</resolution>
+                </range>
+                <noise>
+                    <type>gaussian</type>
+                    <mean>0.0</mean>
+                    <stddev>0.01</stddev>
+                </noise>
+            </ray>
+            <plugin name="scan" filename="libgazebo_ros_ray_sensor.so">
+                <ros>
+                    <remapping>~/out:=scan</remapping>
+                </ros>
+                <output_type>sensor_msgs/LaserScan</output_type>
+                <frame_name>lidar_link</frame_name>
+            </plugin>
+        </sensor>
+    </gazebo>
+    <gazebo reference="camera_link">
+        <sensor type="camera" name="camera1">
+            <update_rate>30.0</update_rate>
+            <camera name="head">
+                <horizontal_fov>1.5127496682368</horizontal_fov>
+                <verical_fov>1.6500906166776</verical_fov>
+                <image>
+                    <width>1280</width>
+                    <height>720</height>
+                    <format>R8G8B8</format>
+                </image>
+                <clip>
+                    <near>0.02</near>
+                    <far>300</far>
+                </clip>
+                <noise>
+                    <type>gaussian</type>
+                    <!-- Noise is sampled independently per pixel on each frame.
+               That pixel's noise value is added to each of its color
+               channels, which at that point lie in the range [0,1]. -->
+                    <mean>0.0</mean>
+                    <stddev>0.007</stddev>
+                </noise>
+            </camera>
+            <plugin name="camera_controller" filename="libgazebo_ros_camera.so">
+                <alwaysOn>true</alwaysOn>
+                <updateRate>0.0</updateRate>
+                <cameraName>drives/camera1</cameraName>
+                <imageTopicName>image_raw</imageTopicName>
+                <cameraInfoTopicName>camera_info</cameraInfoTopicName>
+                <frameName>camera_link</frameName>
+                <hackBaseline>0.07</hackBaseline>
+                <distortionK1>0.0</distortionK1>
+                <distortionK2>0.0</distortionK2>
+                <distortionK3>0.0</distortionK3>
+                <distortionT1>0.0</distortionT1>
+                <distortionT2>0.0</distortionT2>
+            </plugin>
+        </sensor>
+    </gazebo>
 </robot>

Commit message: resolved merge conflicts

File: src/cmr_description/cmr_drives_description/urdf/drives_description.urdf.xacro (robot description, xacro)
@@ -185,4 +185,22 @@
         <xacro:wheel name="right_back" x="-${base_width/2}" y="${base_length/2 + wheel_len}" />
     </xacro:macro>
+    <link name="imu_link">
+        <visual>
+            <geometry>
+                <box size="0.1 0.1 0.1"/>
+            </geometry>
+        </visual>
+        <collision>
+            <geometry>
+                <box size="0.1 0.1 0.1"/>
+            </geometry>
+        </collision>
+        <!-- <xacro:box_inertia m="0.1" w="0.1" d="0.1" h="0.1"/> -->
+    </link>
+    <joint name="imu_joint" type="fixed">
+        <parent link="base_link"/>
+        <child link="imu_link"/>
+        <origin xyz="0 0 0.01"/>
+    </joint>
     <gazebo reference="imu_link">
         <gravity>true</gravity>
@@ -265,20 +283,15 @@
         <plugin name='diff_drive' filename='libgazebo_ros_diff_drive.so'>
             <ros>
-                <namespace>/</namespace>
+                <namespace>/demo</namespace>
             </ros>
             <!-- wheels -->
-            <num_wheel_pairs>3</num_wheel_pairs>
-            <left_joint>left_front_joint</left_joint>
-            <left_joint>left_mid_joint</left_joint>
-            <left_joint>left_back_joint</left_joint>
-            <right_joint>right_front_joint</right_joint>
-            <right_joint>right_mid_joint</right_joint>
-            <right_joint>right_back_joint</right_joint>
+            <left_joint>drivewhl_l_joint</left_joint>
+            <right_joint>drivewhl_r_joint</right_joint>
             <!-- kinematics -->
-            <wheel_separation>0.5</wheel_separation>
+            <wheel_separation>0.4</wheel_separation>
             <wheel_diameter>0.2</wheel_diameter>
             <!-- limits -->
-            <max_wheel_torque>500</max_wheel_torque>
-            <max_wheel_acceleration>10.0</max_wheel_acceleration>
+            <max_wheel_torque>20</max_wheel_torque>
+            <max_wheel_acceleration>1.0</max_wheel_acceleration>
             <!-- output -->
             <update_rate>30</update_rate>
@@ -288,5 +301,4 @@
             <odom_topic>/rover/odom</odom_topic>
             <topic>/cmd_vel</topic>
-            <source_frame>map</source_frame>
             <odometry_frame>odom</odometry_frame>
             <robot_base_frame>base_link</robot_base_frame>
