Commit message: updated urdf to main version Resolved merge conflicts with stephen branch

File: src/cmr_description/cmr_drives_description/urdf/drives_description.urdf.xacro (robot description, xacro)
@@ -61,24 +61,24 @@
                 <min_depth>0.00</min_depth> -->
                 <surface>
-                  <friction>
-                    <ode>
-                      <mu>1.5</mu>
-                      <mu2>1.5</mu2>
-                      <slip1>0</slip1>
-                      <slip2>0</slip2>
-                    </ode>
-                  </friction>
-                   <contact>
-                    <ode>
-                      <soft_cfm>0</soft_cfm>
-                      <soft_erp>0.2</soft_erp>
-                      <kp>1e+13</kp>
-                      <kd>1</kd>
-                      <max_vel>1</max_vel>
-                      <min_depth>0.01</min_depth>
-                    </ode>
-                  </contact>
+                    <friction>
+                        <ode>
+                            <mu>1.5</mu>
+                            <mu2>1.5</mu2>
+                            <slip1>0</slip1>
+                            <slip2>0</slip2>
+                        </ode>
+                    </friction>
+                    <contact>
+                        <ode>
+                            <soft_cfm>0</soft_cfm>
+                            <soft_erp>0.2</soft_erp>
+                            <kp>1e+13</kp>
+                            <kd>1</kd>
+                            <max_vel>1</max_vel>
+                            <min_depth>0.01</min_depth>
+                        </ode>
+                    </contact>
                 </surface>
-              </gazebo>
+            </gazebo>
         </xacro:macro>
         <!-- Base Link -->
@@ -108,10 +108,5 @@
                 <origin xyz="0 0 0" rpy="0 0 0"/>
                 <mass value="${lidar_mass}"/>
-                <inertia ixx="${lidar_mass / 12.0 * (3.0 * lidar_radius * lidar_radius + lidar_height * lidar_height)}"
-                         ixy="0"
-                         ixz="0"
-                         iyy="${lidar_mass / 12.0 * (3.0 * lidar_radius * lidar_radius + lidar_height * lidar_height)}"
-                         iyz="0"
-                         izz="${0.5 * lidar_mass * lidar_radius * lidar_radius}" />
+                <inertia ixx="${lidar_mass / 12.0 * (3.0 * lidar_radius * lidar_radius + lidar_height * lidar_height)}" ixy="0" ixz="0" iyy="${lidar_mass / 12.0 * (3.0 * lidar_radius * lidar_radius + lidar_height * lidar_height)}" iyz="0" izz="${0.5 * lidar_mass * lidar_radius * lidar_radius}" />
             </inertial>
             <collision>
@@ -164,10 +159,5 @@
                 <origin xyz="0 0 0" rpy="0 0 0"/>
                 <mass value="${camera_mass}"/>
-                <inertia ixx="${camera_mass / 12.0 * (cam_height * cam_height + cam_length * cam_length)}"
-                         ixy="0"
-                         ixz="0"
-                         iyy="${camera_mass / 12.0 * (cam_height * cam_height + cam_width * cam_width)}"
-                         iyz="0"
-                         izz="${camera_mass / 12.0 * (cam_width * cam_width + cam_length * cam_length)}" />
+                <inertia ixx="${camera_mass / 12.0 * (cam_height * cam_height + cam_length * cam_length)}" ixy="0" ixz="0" iyy="${camera_mass / 12.0 * (cam_height * cam_height + cam_width * cam_width)}" iyz="0" izz="${camera_mass / 12.0 * (cam_width * cam_width + cam_length * cam_length)}" />
             </inertial>
         </link>
@@ -185,22 +175,4 @@
         <xacro:wheel name="right_back" x="-${base_width/2}" y="${base_length/2 + wheel_len}" />
     </xacro:macro>
-    <link name="imu_link">
-        <visual>
-            <geometry>
-                <box size="0.1 0.1 0.1"/>
-            </geometry>
-        </visual>
-        <collision>
-            <geometry>
-                <box size="0.1 0.1 0.1"/>
-            </geometry>
-        </collision>
-        <!-- <xacro:box_inertia m="0.1" w="0.1" d="0.1" h="0.1"/> -->
-    </link>
-    <joint name="imu_joint" type="fixed">
-        <parent link="base_link"/>
-        <child link="imu_link"/>
-        <origin xyz="0 0 0.01"/>
-    </joint>
     <gazebo reference="imu_link">
         <gravity>true</gravity>
@@ -283,15 +255,20 @@
         <plugin name='diff_drive' filename='libgazebo_ros_diff_drive.so'>
             <ros>
-                <namespace>/demo</namespace>
+                <namespace>/</namespace>
             </ros>
             <!-- wheels -->
-            <left_joint>drivewhl_l_joint</left_joint>
-            <right_joint>drivewhl_r_joint</right_joint>
+            <num_wheel_pairs>3</num_wheel_pairs>
+            <left_joint>left_front_joint</left_joint>
+            <left_joint>left_mid_joint</left_joint>
+            <left_joint>left_back_joint</left_joint>
+            <right_joint>right_front_joint</right_joint>
+            <right_joint>right_mid_joint</right_joint>
+            <right_joint>right_back_joint</right_joint>
             <!-- kinematics -->
-            <wheel_separation>0.4</wheel_separation>
+            <wheel_separation>0.5</wheel_separation>
             <wheel_diameter>0.2</wheel_diameter>
             <!-- limits -->
-            <max_wheel_torque>20</max_wheel_torque>
-            <max_wheel_acceleration>1.0</max_wheel_acceleration>
+            <max_wheel_torque>500</max_wheel_torque>
+            <max_wheel_acceleration>10.0</max_wheel_acceleration>
             <!-- output -->
             <update_rate>30</update_rate>
@@ -301,4 +278,5 @@
             <odom_topic>/rover/odom</odom_topic>
             <topic>/cmd_vel</topic>
+            <source_frame>map</source_frame>
             <odometry_frame>odom</odometry_frame>
             <robot_base_frame>base_link</robot_base_frame>

Commit message: Localization setup, more nav debugging

File: src/cmr_description/cmr_drives_description/urdf/drives_description.urdf.xacro (robot description, xacro)
@@ -22,7 +22,4 @@
         <xacro:property name="cam_height" value="${base_height / 10.0}" />
         <xacro:property name="cam_length" value="${base_length / 10.0}" />
-        <xacro:property name="imu_width" value="${base_width}" />
-        <xacro:property name="imu_height" value="${base_height / 2.0}" />
-        <xacro:property name="imu_length" value="${base_length}" />
         <!-- Space btw top of beam and the each joint -->
         <xacro:macro name="wheel" params="name x y">
@@ -134,35 +131,20 @@
             <parent link="base_link"/>
             <child link="lidar_link"/>
-            <origin xyz="0 0 ${base_height*2}" rpy="0 0 0"/>
+            <origin xyz="0 0 ${base_height}" rpy="0 0 0"/>
         </joint>
         <!-- IMU Link -->
-        <link name="imu_link">
-            <visual>
-                <geometry>
-                    <box size="${imu_width} ${imu_length} ${imu_height}"/>
-                </geometry>
-            </visual>
-            <collision>
-                <geometry>
-                    <box size="${imu_width} ${imu_length} ${imu_height}"/>
-                </geometry>
-            </collision>
-            <!-- <xacro:box_inertia m="0.1" w="0.1" d="0.1" h="0.1"/> -->
-            <inertial>
-                <origin xyz="0 0 0" rpy="0 0 0"/>
-                <mass value="${imu_mass}"/>
-                <inertia ixx="${imu_mass / 12.0 * (imu_height * imu_height + imu_length * imu_length)}"
-                         ixy="0"
-                         ixz="0"
-                         iyy="${imu_mass / 12.0 * (imu_height * imu_height + imu_width * imu_width)}"
-                         iyz="0"
-                         izz="${imu_mass / 12.0 * (imu_width * imu_width + imu_length * imu_length)}" />
-            </inertial>
-        </link>
         <joint name="imu_joint" type="fixed">
             <parent link="base_link"/>
             <child link="imu_link"/>
-            <origin xyz="0 0 ${base_height * 1.25}"/>
+            <origin xyz="0 0 0"/>
         </joint>
+        <link name="imu_link" />
+        <!-- GPS Link -->
+        <joint name="gps_joint" type="fixed">
+            <parent link="base_link"/>
+            <child link="gps_link"/>
+            <origin xyz="0 0 0"/>
+        </joint>
+        <link name="gps_link" />
         <!-- Camera Link -->
         <link name="camera_link">
@@ -193,5 +175,5 @@
             <parent link="base_link"/>
             <child link="camera_link"/>
-            <origin xyz="${base_width / 2} 0 ${base_height}" rpy="0 0 0"/>
+            <origin xyz="${base_width / 2} 0 ${base_height / 2}" rpy="0 0 0"/>
         </joint>
         <!-- Wheels -->
@@ -204,8 +186,9 @@
     </xacro:macro>
     <gazebo reference="imu_link">
+        <gravity>true</gravity>
         <sensor name="imu_sensor" type="imu">
             <plugin filename="libgazebo_ros_imu_sensor.so" name="imu_plugin">
                 <ros>
-                    <namespace>/</namespace>
+                    <namespace>/rover</namespace>
                     <remapping>~/out:=imu</remapping>
                 </ros>
@@ -216,57 +199,65 @@
             <visualize>true</visualize>
             <imu>
+                <orientation>
+                  <x>
+                    <noise type="gaussian">
+                      <mean>0.0</mean>
+                      <stddev>2e-3</stddev>
+                    </noise>
+                  </x>
+                  <y>
+                    <noise type="gaussian">
+                      <mean>0.0</mean>
+                      <stddev>2e-3</stddev>
+                    </noise>
+                  </y>
+                  <z>
+                    <noise type="gaussian">
+                      <mean>0.0</mean>
+                      <stddev>2e-3</stddev>
+                    </noise>
+                  </z>
+                </orientation>
                 <angular_velocity>
-                    <x>
-                        <noise type="gaussian">
-                            <mean>0.0</mean>
-                            <stddev>2e-4</stddev>
-                            <bias_mean>0.0000075</bias_mean>
-                            <bias_stddev>0.0000008</bias_stddev>
-                        </noise>
-                    </x>
-                    <y>
-                        <noise type="gaussian">
-                            <mean>0.0</mean>
-                            <stddev>2e-4</stddev>
-                            <bias_mean>0.0000075</bias_mean>
-                            <bias_stddev>0.0000008</bias_stddev>
-                        </noise>
-                    </y>
-                    <z>
-                        <noise type="gaussian">
-                            <mean>0.0</mean>
-                            <stddev>2e-4</stddev>
-                            <bias_mean>0.0000075</bias_mean>
-                            <bias_stddev>0.0000008</bias_stddev>
-                        </noise>
-                    </z>
+                  <x>
+                    <noise type="gaussian">
+                      <mean>0.0</mean>
+                      <stddev>2e-4</stddev>
+                    </noise>
+                  </x>
+                  <y>
+                    <noise type="gaussian">
+                      <mean>0.0</mean>
+                      <stddev>2e-4</stddev>
+                    </noise>
+                  </y>
+                  <z>
+                    <noise type="gaussian">
+                      <mean>0.0</mean>
+                      <stddev>2e-4</stddev>
+                    </noise>
+                  </z>
                 </angular_velocity>
                 <linear_acceleration>
-                    <x>
-                        <noise type="gaussian">
-                            <mean>0.0</mean>
-                            <stddev>1.7e-2</stddev>
-                            <bias_mean>0.1</bias_mean>
-                            <bias_stddev>0.001</bias_stddev>
-                        </noise>
-                    </x>
-                    <y>
-                        <noise type="gaussian">
-                            <mean>0.0</mean>
-                            <stddev>1.7e-2</stddev>
-                            <bias_mean>0.1</bias_mean>
-                            <bias_stddev>0.001</bias_stddev>
-                        </noise>
-                    </y>
-                    <z>
-                        <noise type="gaussian">
-                            <mean>0.0</mean>
-                            <stddev>1.7e-2</stddev>
-                            <bias_mean>0.1</bias_mean>
-                            <bias_stddev>0.001</bias_stddev>
-                        </noise>
-                    </z>
+                  <x>
+                    <noise type="gaussian">
+                      <mean>0.0</mean>
+                      <stddev>1.7e-2</stddev>
+                    </noise>
+                  </x>
+                  <y>
+                    <noise type="gaussian">
+                      <mean>0.0</mean>
+                      <stddev>1.7e-2</stddev>
+                    </noise>
+                  </y>
+                  <z>
+                    <noise type="gaussian">
+                      <mean>0.0</mean>
+                      <stddev>1.7e-2</stddev>
+                    </noise>
+                  </z>
                 </linear_acceleration>
-            </imu>
+              </imu>
         </sensor>
     </gazebo>
@@ -291,9 +282,9 @@
             <max_wheel_acceleration>10.0</max_wheel_acceleration>
             <!-- output -->
-            <odom_publish_frequency>1</odom_publish_frequency>
+            <update_rate>30</update_rate>
             <publish_odom>true</publish_odom>
-            <publish_odom_tf>true</publish_odom_tf>
-            <publish_wheel_tf>true</publish_wheel_tf>
-            <odom_topic>/odom</odom_topic>
+            <publish_odom_tf>false</publish_odom_tf>
+            <publish_wheel_tf>false</publish_wheel_tf>
+            <odom_topic>/rover/odom</odom_topic>
             <topic>/cmd_vel</topic>
             <source_frame>map</source_frame>
@@ -317,6 +308,6 @@
                 </scan>
                 <range>
-                    <min>0.120000</min>
-                    <max>3.5</max>
+                    <min>0.150000</min>
+                    <max>12.0</max>
                     <resolution>0.015000</resolution>
                 </range>
@@ -376,3 +367,30 @@
         </sensor>
     </gazebo>
+    <gazebo reference="gps_link">
+        <sensor name="rover_gps" type="gps">
+            <always_on>true</always_on>
+            <update_rate>10.0</update_rate>
+            <gps>
+            <position_sensing>
+                <horizontal>
+                <noise type="gaussian">
+                    <mean>0.0</mean>
+                    <stddev>1e-2</stddev>
+                </noise>
+                </horizontal>
+                <vertical>
+                <noise type="gaussian">
+                    <mean>0.0</mean>
+                    <stddev>1</stddev>
+                </noise>
+                </vertical>
+            </position_sensing>
+            </gps>
+            <plugin name="rover_gps" filename="libgazebo_ros_gps_sensor.so">
+            <ros>
+                <remapping>~/out:=gps/fix</remapping>
+            </ros>
+            </plugin>
+        </sensor>
+    </gazebo>
 </robot>
