Commit message: A little better

File: src/cmr_description/cmr_drives_description/urdf/drives_description.urdf.xacro (robot description, xacro)
@@ -61,24 +61,24 @@
                 <min_depth>0.00</min_depth> -->
                 <surface>
-                  <friction>
-                    <ode>
-                      <mu>1.5</mu>
-                      <mu2>1.5</mu2>
-                      <slip1>0</slip1>
-                      <slip2>0</slip2>
-                    </ode>
-                  </friction>
-                   <contact>
-                    <ode>
-                      <soft_cfm>0</soft_cfm>
-                      <soft_erp>0.2</soft_erp>
-                      <kp>1e+13</kp>
-                      <kd>1</kd>
-                      <max_vel>1</max_vel>
-                      <min_depth>0.01</min_depth>
-                    </ode>
-                  </contact>
+                    <friction>
+                        <ode>
+                            <mu>1.5</mu>
+                            <mu2>1.5</mu2>
+                            <slip1>0</slip1>
+                            <slip2>0</slip2>
+                        </ode>
+                    </friction>
+                    <contact>
+                        <ode>
+                            <soft_cfm>0</soft_cfm>
+                            <soft_erp>0.2</soft_erp>
+                            <kp>1e+13</kp>
+                            <kd>1</kd>
+                            <max_vel>1</max_vel>
+                            <min_depth>0.01</min_depth>
+                        </ode>
+                    </contact>
                 </surface>
-              </gazebo>
+            </gazebo>
         </xacro:macro>
         <!-- Base Link -->
@@ -108,10 +108,5 @@
                 <origin xyz="0 0 0" rpy="0 0 0"/>
                 <mass value="${lidar_mass}"/>
-                <inertia ixx="${lidar_mass / 12.0 * (3.0 * lidar_radius * lidar_radius + lidar_height * lidar_height)}"
-                         ixy="0"
-                         ixz="0"
-                         iyy="${lidar_mass / 12.0 * (3.0 * lidar_radius * lidar_radius + lidar_height * lidar_height)}"
-                         iyz="0"
-                         izz="${0.5 * lidar_mass * lidar_radius * lidar_radius}" />
+                <inertia ixx="${lidar_mass / 12.0 * (3.0 * lidar_radius * lidar_radius + lidar_height * lidar_height)}" ixy="0" ixz="0" iyy="${lidar_mass / 12.0 * (3.0 * lidar_radius * lidar_radius + lidar_height * lidar_height)}" iyz="0" izz="${0.5 * lidar_mass * lidar_radius * lidar_radius}" />
             </inertial>
             <collision>
@@ -164,10 +159,5 @@
                 <origin xyz="0 0 0" rpy="0 0 0"/>
                 <mass value="${camera_mass}"/>
-                <inertia ixx="${camera_mass / 12.0 * (cam_height * cam_height + cam_length * cam_length)}"
-                         ixy="0"
-                         ixz="0"
-                         iyy="${camera_mass / 12.0 * (cam_height * cam_height + cam_width * cam_width)}"
-                         iyz="0"
-                         izz="${camera_mass / 12.0 * (cam_width * cam_width + cam_length * cam_length)}" />
+                <inertia ixx="${camera_mass / 12.0 * (cam_height * cam_height + cam_length * cam_length)}" ixy="0" ixz="0" iyy="${camera_mass / 12.0 * (cam_height * cam_height + cam_width * cam_width)}" iyz="0" izz="${camera_mass / 12.0 * (cam_width * cam_width + cam_length * cam_length)}" />
             </inertial>
         </link>
@@ -200,64 +190,64 @@
             <imu>
                 <orientation>
-                  <x>
-                    <noise type="gaussian">
-                      <mean>0.0</mean>
-                      <stddev>2e-3</stddev>
-                    </noise>
-                  </x>
-                  <y>
-                    <noise type="gaussian">
-                      <mean>0.0</mean>
-                      <stddev>2e-3</stddev>
-                    </noise>
-                  </y>
-                  <z>
-                    <noise type="gaussian">
-                      <mean>0.0</mean>
-                      <stddev>2e-3</stddev>
-                    </noise>
-                  </z>
+                    <x>
+                        <noise type="gaussian">
+                            <mean>0.0</mean>
+                            <stddev>2e-3</stddev>
+                        </noise>
+                    </x>
+                    <y>
+                        <noise type="gaussian">
+                            <mean>0.0</mean>
+                            <stddev>2e-3</stddev>
+                        </noise>
+                    </y>
+                    <z>
+                        <noise type="gaussian">
+                            <mean>0.0</mean>
+                            <stddev>2e-3</stddev>
+                        </noise>
+                    </z>
                 </orientation>
                 <angular_velocity>
-                  <x>
-                    <noise type="gaussian">
-                      <mean>0.0</mean>
-                      <stddev>2e-4</stddev>
-                    </noise>
-                  </x>
-                  <y>
-                    <noise type="gaussian">
-                      <mean>0.0</mean>
-                      <stddev>2e-4</stddev>
-                    </noise>
-                  </y>
-                  <z>
-                    <noise type="gaussian">
-                      <mean>0.0</mean>
-                      <stddev>2e-4</stddev>
-                    </noise>
-                  </z>
+                    <x>
+                        <noise type="gaussian">
+                            <mean>0.0</mean>
+                            <stddev>2e-4</stddev>
+                        </noise>
+                    </x>
+                    <y>
+                        <noise type="gaussian">
+                            <mean>0.0</mean>
+                            <stddev>2e-4</stddev>
+                        </noise>
+                    </y>
+                    <z>
+                        <noise type="gaussian">
+                            <mean>0.0</mean>
+                            <stddev>2e-4</stddev>
+                        </noise>
+                    </z>
                 </angular_velocity>
                 <linear_acceleration>
-                  <x>
-                    <noise type="gaussian">
-                      <mean>0.0</mean>
-                      <stddev>1.7e-2</stddev>
-                    </noise>
-                  </x>
-                  <y>
-                    <noise type="gaussian">
-                      <mean>0.0</mean>
-                      <stddev>1.7e-2</stddev>
-                    </noise>
-                  </y>
-                  <z>
-                    <noise type="gaussian">
-                      <mean>0.0</mean>
-                      <stddev>1.7e-2</stddev>
-                    </noise>
-                  </z>
+                    <x>
+                        <noise type="gaussian">
+                            <mean>0.0</mean>
+                            <stddev>1.7e-2</stddev>
+                        </noise>
+                    </x>
+                    <y>
+                        <noise type="gaussian">
+                            <mean>0.0</mean>
+                            <stddev>1.7e-2</stddev>
+                        </noise>
+                    </y>
+                    <z>
+                        <noise type="gaussian">
+                            <mean>0.0</mean>
+                            <stddev>1.7e-2</stddev>
+                        </noise>
+                    </z>
                 </linear_acceleration>
-              </imu>
+            </imu>
         </sensor>
     </gazebo>
@@ -286,5 +276,5 @@
             <publish_odom_tf>true</publish_odom_tf>
             <publish_wheel_tf>false</publish_wheel_tf>
-            <odom_topic>/rover/odom</odom_topic>
+            <odom_topic>/odom</odom_topic>
             <topic>/cmd_vel</topic>
             <source_frame>map</source_frame>
@@ -297,5 +287,5 @@
             <always_on>true</always_on>
             <visualize>true</visualize>
-            <update_rate>5</update_rate>
+            <update_rate>20</update_rate>
             <ray>
                 <scan>
@@ -372,23 +362,23 @@
             <update_rate>10.0</update_rate>
             <gps>
-            <position_sensing>
-                <horizontal>
-                <noise type="gaussian">
-                    <mean>0.0</mean>
-                    <stddev>1e-2</stddev>
-                </noise>
-                </horizontal>
-                <vertical>
-                <noise type="gaussian">
-                    <mean>0.0</mean>
-                    <stddev>1</stddev>
-                </noise>
-                </vertical>
-            </position_sensing>
+                <position_sensing>
+                    <horizontal>
+                        <noise type="gaussian">
+                            <mean>0.0</mean>
+                            <stddev>1e-2</stddev>
+                        </noise>
+                    </horizontal>
+                    <vertical>
+                        <noise type="gaussian">
+                            <mean>0.0</mean>
+                            <stddev>1</stddev>
+                        </noise>
+                    </vertical>
+                </position_sensing>
             </gps>
             <plugin name="rover_gps" filename="libgazebo_ros_gps_sensor.so">
-            <ros>
-                <remapping>~/out:=gps/fix</remapping>
-            </ros>
+                <ros>
+                    <remapping>~/out:=gps/fix</remapping>
+                </ros>
             </plugin>
         </sensor>

Commit message: More tests

File: src/cmr_description/cmr_drives_description/urdf/drives_description.urdf.xacro (robot description, xacro)
@@ -123,8 +123,9 @@
             </visual>
         </link>
-        <joint name="lidar_joint" type="fixed">
+        <joint name="lidar_joint" type="continuous">
             <parent link="base_link"/>
             <child link="lidar_link"/>
             <origin xyz="0 0 ${base_height}" rpy="0 0 0"/>
+            <axis xyz="0 1 0" />
         </joint>
         <!-- IMU Link -->

Commit message: Add turtlebot3

File: src/cmr_description/cmr_drives_description/urdf/drives_description.urdf.xacro (robot description, xacro)
@@ -123,9 +123,8 @@
             </visual>
         </link>
-        <joint name="lidar_joint" type="continuous">
+        <joint name="lidar_joint" type="fixed">
             <parent link="base_link"/>
             <child link="lidar_link"/>
             <origin xyz="0 0 ${base_height}" rpy="0 0 0"/>
-            <axis xyz="0 1 0" />
         </joint>
         <!-- IMU Link -->

Commit message: Add base_footprint

File: src/cmr_description/cmr_drives_description/urdf/drives_description.urdf.xacro (robot description, xacro)
@@ -82,4 +82,10 @@
             </gazebo>
         </xacro:macro>
+        <link name="base_footprint"/>
+        <joint name="base_joint" type="fixed">
+            <parent link="base_footprint"/>
+            <child link="base_link" />
+            <origin xyz="0 0 0.010" rpy="0 0 0"/>
+        </joint>
         <!-- Base Link -->
         <link name="base_link">
