Commit message: Update arm configuration for joystick control

File: src/cmr_arm_config/config/arm.ros2_control.xacro (robot description, xacro)
@@ -1,61 +1,61 @@
 <?xml version="1.0"?>
 <robot xmlns:xacro="http://www.ros.org/wiki/xacro">
-    <xacro:macro name="arm_ros2_control" params="name initial_positions_file">
-        <xacro:property name="initial_positions" value="${load_yaml(initial_positions_file)['initial_positions']}"/>
-        <ros2_control name="${name}" type="system">
-            <hardware>
-                <!-- By default, set up controllers for simulation. This won't work on real hardware -->
-                <plugin>mock_components/GenericSystem</plugin>
-            </hardware>
-            <joint name="base_rotate">
-                <command_interface name="position"/>
-                <state_interface name="position">
-                  <param name="initial_value">${initial_positions['base_rotate']}</param>
-                </state_interface>
-                <state_interface name="velocity"/>
-            </joint>
-            <joint name="shoulder">
-                <command_interface name="position"/>
-                <state_interface name="position">
-                  <param name="initial_value">${initial_positions['shoulder']}</param>
-                </state_interface>
-                <state_interface name="velocity"/>
-            </joint>
-            <joint name="elbow">
-                <command_interface name="position"/>
-                <state_interface name="position">
-                  <param name="initial_value">${initial_positions['elbow']}</param>
-                </state_interface>
-                <state_interface name="velocity"/>
-            </joint>
-            <joint name="second_rotate">
-                <command_interface name="position"/>
-                <state_interface name="position">
-                  <param name="initial_value">${initial_positions['second_rotate']}</param>
-                </state_interface>
-                <state_interface name="velocity"/>
-            </joint>
-            <joint name="third_tilt">
-                <command_interface name="position"/>
-                <state_interface name="position">
-                  <param name="initial_value">${initial_positions['third_tilt']}</param>
-                </state_interface>
-                <state_interface name="velocity"/>
-            </joint>
-            <joint name="third_rotate">
-                <command_interface name="position"/>
-                <state_interface name="position">
-                  <param name="initial_value">${initial_positions['third_rotate']}</param>
-                </state_interface>
-                <state_interface name="velocity"/>
-            </joint>
-            <joint name="end_effector">
-                <command_interface name="position"/>
-                <state_interface name="position">
-                  <param name="initial_value">${initial_positions['end_effector']}</param>
-                </state_interface>
-                <state_interface name="velocity"/>
-            </joint>
-        </ros2_control>
-    </xacro:macro>
+  <xacro:macro name="arm_ros2_control" params="name initial_positions_file">
+    <xacro:property name="initial_positions" value="${load_yaml(initial_positions_file)['initial_positions']}"/>
+    <ros2_control name="${name}" type="system">
+      <hardware>
+        <!-- By default, set up controllers for simulation. This won't work on real hardware -->
+        <plugin>mock_components/GenericSystem</plugin>
+      </hardware>
+      <joint name="base_rotate">
+        <command_interface name="position"/>
+        <state_interface name="position">
+          <param name="initial_value">${initial_positions['base_rotate']}</param>
+        </state_interface>
+        <state_interface name="velocity"/>
+      </joint>
+      <joint name="shoulder">
+        <command_interface name="position"/>
+        <state_interface name="position">
+          <param name="initial_value">${initial_positions['shoulder']}</param>
+        </state_interface>
+        <state_interface name="velocity"/>
+      </joint>
+      <joint name="elbow">
+        <command_interface name="position"/>
+        <state_interface name="position">
+          <param name="initial_value">${initial_positions['elbow']}</param>
+        </state_interface>
+        <state_interface name="velocity"/>
+      </joint>
+      <joint name="second_rotate">
+        <command_interface name="position"/>
+        <state_interface name="position">
+          <param name="initial_value">${initial_positions['second_rotate']}</param>
+        </state_interface>
+        <state_interface name="velocity"/>
+      </joint>
+      <joint name="third_tilt">
+        <command_interface name="position"/>
+        <state_interface name="position">
+          <param name="initial_value">${initial_positions['third_tilt']}</param>
+        </state_interface>
+        <state_interface name="velocity"/>
+      </joint>
+      <joint name="third_rotate">
+        <command_interface name="position"/>
+        <state_interface name="position">
+          <param name="initial_value">${initial_positions['third_rotate']}</param>
+        </state_interface>
+        <state_interface name="velocity"/>
+      </joint>
+      <joint name="end_effector">
+        <command_interface name="position"/>
+        <state_interface name="position">
+          <param name="initial_value">${initial_positions['end_effector']}</param>
+        </state_interface>
+        <state_interface name="velocity"/>
+      </joint>
+    </ros2_control>
+  </xacro:macro>
 </robot>

File: src/cmr_description/cmr_arm_description/ros2_control/arm.ros2_control.xacro (robot description, xacro)
@@ -13,5 +13,5 @@
             <joint name="base_rotate">
                 <command_interface name="position"/>
-                <command_interface name="effort"/>
+                <command_interface name="velocity"/>
                 <state_interface name="position"/>
                 <state_interface name="velocity"/>
@@ -19,5 +19,5 @@
             <joint name="shoulder">
                 <command_interface name="position"/>
-                <command_interface name="effort"/>
+                <command_interface name="velocity"/>
                 <state_interface name="position"/>
                 <state_interface name="velocity"/>
@@ -25,5 +25,5 @@
             <joint name="elbow">
                 <command_interface name="position"/>
-                <command_interface name="effort"/>
+                <command_interface name="velocity"/>
                 <state_interface name="position"/>
                 <state_interface name="velocity"/>
@@ -31,5 +31,5 @@
             <joint name="second_rotate">
                 <command_interface name="position"/>
-                <command_interface name="effort"/>
+                <command_interface name="velocity"/>
                 <state_interface name="position"/>
                 <state_interface name="velocity"/>
@@ -37,5 +37,5 @@
             <joint name="third_tilt">
                 <command_interface name="position"/>
-                <command_interface name="effort"/>
+                <command_interface name="velocity"/>
                 <state_interface name="position"/>
                 <state_interface name="velocity"/>
@@ -43,5 +43,5 @@
             <joint name="third_rotate">
                 <command_interface name="position"/>
-                <command_interface name="effort"/>
+                <command_interface name="velocity"/>
                 <state_interface name="position"/>
                 <state_interface name="velocity"/>

Commit message: Updated URDF (needs fixing)

File: src/cmr_arm_config/config/arm.ros2_control.xacro (robot description, xacro)
@@ -8,50 +8,49 @@
         <plugin>mock_components/GenericSystem</plugin>
       </hardware>
-      <joint name="base_rotate">
+      <!-- Joint "base_joint" -->
+      <joint name="base_joint">
         <command_interface name="position"/>
         <state_interface name="position">
-          <param name="initial_value">${initial_positions['base_rotate']}</param>
+          <param name="initial_value">${initial_positions['base_joint']}</param>
         </state_interface>
         <state_interface name="velocity"/>
       </joint>
-      <joint name="shoulder">
+      <!-- Joint "shoulder_joint" -->
+      <joint name="shoulder_joint">
         <command_interface name="position"/>
         <state_interface name="position">
-          <param name="initial_value">${initial_positions['shoulder']}</param>
+          <param name="initial_value">${initial_positions['shoulder_joint']}</param>
         </state_interface>
         <state_interface name="velocity"/>
       </joint>
-      <joint name="elbow">
+      <!-- Joint "elbow_joint" -->
+      <joint name="elbow_joint">
         <command_interface name="position"/>
         <state_interface name="position">
-          <param name="initial_value">${initial_positions['elbow']}</param>
+          <param name="initial_value">${initial_positions['elbow_joint']}</param>
         </state_interface>
         <state_interface name="velocity"/>
       </joint>
-      <joint name="second_rotate">
+      <!-- Joint "wrist_rotate" -->
+      <joint name="wrist_rotate">
         <command_interface name="position"/>
         <state_interface name="position">
-          <param name="initial_value">${initial_positions['second_rotate']}</param>
+          <param name="initial_value">${initial_positions['wrist_rotate']}</param>
         </state_interface>
         <state_interface name="velocity"/>
       </joint>
-      <joint name="third_tilt">
+      <!-- Joint "wrist_twist" -->
+      <joint name="wrist_twist">
         <command_interface name="position"/>
         <state_interface name="position">
-          <param name="initial_value">${initial_positions['third_tilt']}</param>
+          <param name="initial_value">${initial_positions['wrist_twist']}</param>
         </state_interface>
         <state_interface name="velocity"/>
       </joint>
-      <joint name="third_rotate">
+      <!-- Joint "wrist_rotate_two" -->
+      <joint name="wrist_rotate_two">
         <command_interface name="position"/>
         <state_interface name="position">
-          <param name="initial_value">${initial_positions['third_rotate']}</param>
-        </state_interface>
-        <state_interface name="velocity"/>
-      </joint>
-      <joint name="end_effector">
-        <command_interface name="position"/>
-        <state_interface name="position">
-          <param name="initial_value">${initial_positions['end_effector']}</param>
+          <param name="initial_value">${initial_positions['wrist_rotate_two']}</param>
         </state_interface>
         <state_interface name="velocity"/>

File: src/cmr_arm_config/config/arm.urdf.xacro (robot description, xacro)
@@ -3,5 +3,5 @@
     <xacro:arg name="initial_positions_file" default="initial_positions.yaml" />
     <!-- Import arm urdf file -->
-    <xacro:include filename="$(find cmr_arm_description)/urdf/arm_no_control.urdf.xacro" />
+    <xacro:include filename="$(find cmr_arm_description)/urdf/arm_2024.urdf.xacro" />
     <!-- Import control_xacro -->
     <xacro:include filename="arm.ros2_control.xacro" />
