Commit message: testing drive to coord on real rover

File: src/rover_description/urdf/include/robot_parts/chassis.xacro (robot description, xacro)
@@ -11,7 +11,7 @@
     <link name="${name}">
       <inertial>
-        <mass value="250"/>
+        <mass value="500"/>
         <origin xyz="0 0 -0.3"/>
-        <inertia ixx="4.368270834" ixy="0" ixz="0" iyy="8.22579" iyz="0" izz="11.62632083"/>
+        <inertia ixx="8.736541668" ixy="0" ixz="0" iyy="16.45158" iyz="0" izz="23.25264166" />
       </inertial>
       <visual>

File: src/rover_description/urdf/include/robot_parts/swerves.xacro (robot description, xacro)
@@ -7,5 +7,5 @@
       <inertial>
         <mass value="1"/>
-        <origin xyz="0 0 0"/>
+        <origin xyz="${x} ${y} ${z}"/>
         <inertia ixx="0.0009375" ixy="0" ixz="0" iyy="0.0009375" iyz="0" izz="0.0009375"/>
       </inertial>

File: src/rover_description/urdf/include/robot_parts/wheels.xacro (robot description, xacro)
@@ -25,4 +25,17 @@
           <cylinder radius="${wheel_radius}" length="${wheel_length}"/>
         </geometry>
+        <surface>
+            <friction>
+            <ode>
+                <mu>0.8</mu>
+                <mu2>0.8</mu2>
+            </ode>
+            </friction>
+            <contact>
+            <ode>
+                <min_depth>0.003</min_depth>
+            </ode>
+            </contact>
+        </surface>
       </collision>
     </link>
@@ -33,5 +46,5 @@
       <axis xyz="0 1 0"/>
       <limit effort="2.0" velocity="27.0"/>
-      <dynamics damping="0.2" friction="0.05"/>
+      <dynamics damping="0.2" friction="0.1"/>
     </joint>
   </xacro:macro>

File: src/rover_description/urdf/include/sensors/depth_camera_sensor.xacro (robot description, xacro)
@@ -30,10 +30,10 @@
         <image>
           <width>640</width>
-          <height>480</height>]
+          <height>480</height>
           <format>R8G8B8</format>
         </image>
         <clip>
           <near>0.3</near>
-          <far>15.0</far>
+          <far>10.0</far>
         </clip>
       </camera>

Commit message: Testing pushing from my github account on team laptop

File: src/rover_description/urdf/include/robot_parts/chassis.xacro (robot description, xacro)
@@ -11,7 +11,7 @@
     <link name="${name}">
       <inertial>
-        <mass value="500"/>
+        <mass value="50"/>
         <origin xyz="0 0 -0.3"/>
-        <inertia ixx="8.736541668" ixy="0" ixz="0" iyy="16.45158" iyz="0" izz="23.25264166" />
+        <inertia ixx="0.8736541668" ixy="0" ixz="0" iyy="1.645158" iyz="0" izz="2.325264166" />
       </inertial>
       <visual>

File: src/rover_description/urdf/include/robot_parts/wheels.xacro (robot description, xacro)
@@ -28,11 +28,11 @@
             <friction>
             <ode>
-                <mu>0.8</mu>
-                <mu2>0.8</mu2>
+                <mu>1.0</mu>
+                <mu2>1.0</mu2>
             </ode>
             </friction>
             <contact>
             <ode>
-                <min_depth>0.003</min_depth>
+                <min_depth>0.05</min_depth>
             </ode>
             </contact>
@@ -45,5 +45,5 @@
       <origin xyz="0 0 0" rpy="0 0 0"/>
       <axis xyz="0 1 0"/>
-      <limit effort="2.0" velocity="27.0"/>
+      <limit effort="1000.0" velocity="27.0"/>
       <dynamics damping="0.2" friction="0.1"/>
     </joint>

File: src/rover_description/urdf/include/sensors/depth_camera_sensor.xacro (robot description, xacro)
@@ -24,5 +24,5 @@
   <gazebo reference="camera_link">
     <sensor type="depth" name="camera">
-      <update_rate>10.0</update_rate>
+      <update_rate>5.0</update_rate>
       <camera>
         <pose>0 0 0 0 0 0</pose>

File: src/rover_description/urdf/include/sensors/gps_sensor.xacro (robot description, xacro)
@@ -17,5 +17,5 @@
                 <noise type="gaussian">
                 <mean>0.0</mean>
-                <stddev>0.01</stddev>
+                <stddev>0.1</stddev>
                 </noise>
             </horizontal>
@@ -23,5 +23,5 @@
                 <noise type="gaussian">
                 <mean>0.0</mean>
-                <stddev>0.01</stddev>
+                <stddev>0.1</stddev>
                 </noise>
             </vertical>
