Commit message: Path planning with A*

File: src/rover_description/urdf/include/sensors/depth_camera_sensor.xacro (robot description, xacro)
@@ -9,5 +9,5 @@
     </visual>
   </link>
-  <joint name="camera_link_joint" type="fixed">
+  <joint name="camera_joint" type="fixed">
     <origin rpy="0 0 0" xyz="0.0 0.0 0.5" />
     <parent link="base_link" />
@@ -15,14 +15,13 @@
     <axis xyz="0 0 0" />
   </joint>
-  <link name="camera_link_frame"></link>
-  <joint name="camera_frame_joint" type="fixed">
-    <origin xyz="0 0 0" rpy="-1.5708 0 -1.5708" />
-    <parent link="camera_link" />
-    <child link="camera_link_frame" />
-    <axis xyz="0 0 0" />
+  <link name="camera_depth_frame"/>
+  <joint name="camera_depth_joint" type="fixed">
+    <origin xyz="0 0 0" rpy="${-pi/2} 0 ${-pi/2}"/>
+    <parent link="camera_link"/>
+    <child link="camera_depth_frame"/>
   </joint>
   <gazebo reference="camera_link">
     <sensor type="depth" name="camera">
-      <update_rate>5.0</update_rate>
+      <update_rate>10.0</update_rate>
       <camera>
         <pose>0 0 0 0 0 0</pose>
@@ -39,5 +38,5 @@
       </camera>
       <plugin name="camera_controller" filename="libgazebo_ros_camera.so">
-        <frame_name>camera_link_frame</frame_name>
+        <frame_name>camera_depth_frame</frame_name>
       </plugin>
     </sensor>

File: src/rover_description/urdf/include/sensors/imu_sensor.xacro (robot description, xacro)
@@ -16,5 +16,5 @@
             </plugin>
             <always_on>true</always_on>
-            <update_rate>100</update_rate>
+            <update_rate>50</update_rate>
             <visualize>true</visualize>
             <imu>
@@ -51,5 +51,5 @@
                         <stddev>1.7e-2</stddev>
                         <bias_mean>0.1</bias_mean>
-                        <bias_stddev>0.001</bias_stddev>
+                        <bias_stddev>0.00001</bias_stddev>
                     </noise>
                     </x>
@@ -59,5 +59,5 @@
                         <stddev>1.7e-2</stddev>
                         <bias_mean>0.1</bias_mean>
-                        <bias_stddev>0.001</bias_stddev>
+                        <bias_stddev>0.00001</bias_stddev>
                     </noise>
                     </y>
@@ -67,5 +67,5 @@
                         <stddev>1.7e-2</stddev>
                         <bias_mean>0.1</bias_mean>
-                        <bias_stddev>0.001</bias_stddev>
+                        <bias_stddev>0.00001</bias_stddev>
                     </noise>
                     </z>

File: src/rover_description/urdf/rover.xacro (robot description, xacro)
@@ -9,3 +9,5 @@
   <xacro:include filename="$(find rover_description)/urdf/include/sensors/gps_sensor.xacro" />
   <xacro:include filename="$(find rover_description)/urdf/include/sensors/imu_sensor.xacro" />
+  <!--Including exact GPS so don't have to worry about localization in sim-->
+  <xacro:include filename="$(find rover_description)/urdf/include/sensors/gps_exact.xacro" />
 </robot>

Commit message: ukf working in sim

File: src/rover_description/urdf/include/sensors/depth_camera_sensor.xacro (robot description, xacro)
@@ -10,5 +10,5 @@
   </link>
   <joint name="camera_joint" type="fixed">
-    <origin rpy="0 0 0" xyz="0.0 0.0 0.5" />
+    <origin rpy="0 0 0" xyz="0.26 0.0 0.5" />
     <parent link="base_link" />
     <child link="camera_link" />

File: src/rover_description/urdf/include/sensors/gps_exact.xacro (robot description, xacro)
@@ -5,5 +5,5 @@
         <parent link="base_link"/>
         <child link="exact_gps" />
-        <origin xyz="0 0 1.0" rpy="0 0 0"/>
+        <origin xyz="0.26 0.08 1.0" rpy="0 0 0"/>
     </joint>
     <gazebo reference="exact_gps">

File: src/rover_description/urdf/include/sensors/imu_sensor.xacro (robot description, xacro)
@@ -5,5 +5,5 @@
         <parent link="base_link"/>
         <child link="imu_link"/>
-        <origin xyz="0 0 0.01"/>
+        <origin xyz="-0.2 0.05 0.01"/>
     </joint>
     <gazebo reference="imu_link">
