Commit message: Update Gazebo rover sim drive path

File: drives.urdf (robot description, URDF)
Before this commit: robot drives, 7 links, 6 joints
Links:
- removed link left_back
- removed link left_front
- removed link left_mid
- removed link right_back
- removed link right_front
- removed link right_mid
- link base_link: mass 0.3 -> 45.0; geometry collision box size=1.08 0.50 0.34; visual mesh filename=file:///cmr/terra2/meshes/rover_26.stl scale=0.001 0.001 0.001
Joints:
- removed joint left_back_joint
- removed joint left_front_joint
- removed joint left_mid_joint
- removed joint right_back_joint
- removed joint right_front_joint
- removed joint right_mid_joint

Commit message: Fix Gazebo rover mesh orientation

File: drives.urdf (robot description, URDF)
Before this commit: robot drives, 1 links, 0 joints
Links:
- link base_link: geometry collision box size=1.08 1.14 0.34; visual mesh filename=file:///cmr/terra2/meshes/rover_26.stl scale=0.001 0.001 0.001

Commit message: Add jointed swerve Gazebo rover model

File: drives.urdf (robot description, URDF)
Before this commit: robot drives, 1 links, 0 joints
Links:
- added link back_left_steer_link, mass 0.5; visual box size=0.08 0.08 0.09
- added link back_left_wheel_link, mass 0.6; visual cylinder length=0.07 radius=0.13
- added link back_right_steer_link, mass 0.5; visual box size=0.08 0.08 0.09
- added link back_right_wheel_link, mass 0.6; visual cylinder length=0.07 radius=0.13
- added link front_left_steer_link, mass 0.5; visual box size=0.08 0.08 0.09
- added link front_left_wheel_link, mass 0.6; visual cylinder length=0.07 radius=0.13
- added link front_right_steer_link, mass 0.5; visual box size=0.08 0.08 0.09
- added link front_right_wheel_link, mass 0.6; visual cylinder length=0.07 radius=0.13
- link base_link: geometry collision box size=0.92 1.00 0.20; visual box size=0.90 0.98 0.18
Joints:
- added joint back_left_steer_joint: type continuous, parent base_link, child back_left_steer_link, origin xyz=-0.415 0.415 0.13 rpy=0 0 0, axis 0 0 1
- added joint back_left_wheel_joint: type continuous, parent back_left_steer_link, child back_left_wheel_link, origin xyz=0 0 0 rpy=0 0 0, axis 0 1 0
- added joint back_right_steer_joint: type continuous, parent base_link, child back_right_steer_link, origin xyz=-0.415 -0.415 0.13 rpy=0 0 0, axis 0 0 1
- added joint back_right_wheel_joint: type continuous, parent back_right_steer_link, child back_right_wheel_link, origin xyz=0 0 0 rpy=0 0 0, axis 0 1 0
- added joint front_left_steer_joint: type continuous, parent base_link, child front_left_steer_link, origin xyz=0.415 0.415 0.13 rpy=0 0 0, axis 0 0 1
- added joint front_left_wheel_joint: type continuous, parent front_left_steer_link, child front_left_wheel_link, origin xyz=0 0 0 rpy=0 0 0, axis 0 1 0
- added joint front_right_steer_joint: type continuous, parent base_link, child front_right_steer_link, origin xyz=0.415 -0.415 0.13 rpy=0 0 0, axis 0 0 1
- added joint front_right_wheel_joint: type continuous, parent front_right_steer_link, child front_right_wheel_link, origin xyz=0 0 0 rpy=0 0 0, axis 0 1 0
