Commit message: Fixed arm urdf display

File: src/cmr_arm_sim/urdf/arm_2024.urdf (robot description, URDF)
Before this commit: robot Arm, 7 links, 6 joints
Links:
- link base_link: geometry collision mesh filename=package://cmr_arm_sim/meshes/base_link.stl scale=1 1 1; visual mesh filename=package://cmr_arm_sim/meshes/base_link.stl scale=1 1 1
- link end_effector: geometry collision mesh filename=package://cmr_arm_sim/meshes/end_effector.stl scale=.039 .039 .039; visual mesh filename=package://cmr_arm_sim/meshes/end_effector.stl scale=.039 .039 .039
- link lower_arm: geometry collision mesh filename=package://cmr_arm_sim/meshes/lower_arm.stl scale=1 1 1; visual mesh filename=package://cmr_arm_sim/meshes/lower_arm.stl scale=1 1 1
- link shoulder: geometry collision mesh filename=package://cmr_arm_sim/meshes/shoulder.stl scale=1 1 1; visual mesh filename=package://cmr_arm_sim/meshes/shoulder.stl scale=1 1 1
- link upper_arm: geometry collision mesh filename=package://cmr_arm_sim/meshes/upper_arm.stl scale=1 1 1; visual mesh filename=package://cmr_arm_sim/meshes/upper_arm.stl scale=1 1 1
- link wrist_rotate: geometry collision mesh filename=package://cmr_arm_sim/meshes/wrist_rotate.stl scale=1 1 1; visual mesh filename=package://cmr_arm_sim/meshes/wrist_rotate.stl scale=1 1 1
- link wrist_twist_rotate: geometry collision mesh filename=package://cmr_arm_sim/meshes/wrist_twist_rotate.stl scale=1 1 1; visual mesh filename=package://cmr_arm_sim/meshes/wrist_twist_rotate.stl scale=1 1 1

Commit message: Added moveit arm sim for the 2024 arm

File: src/cmr_arm_sim/urdf/arm_2024.urdf (robot description, URDF)
Before this commit: robot Arm, 7 links, 6 joints
Links:
- link base_link: geometry collision mesh filename=package://cmr_arm_sim/meshes/base_link.stl scale=0.1 0.1 0.1; visual mesh filename=package://cmr_arm_sim/meshes/base_link.stl scale=0.1 0.1 0.1
- link end_effector: geometry collision mesh filename=package://cmr_arm_sim/meshes/end_effector.stl scale=.0039 .0039 .0039; visual mesh filename=package://cmr_arm_sim/meshes/end_effector.stl scale=.0039 .0039 .0039
- link lower_arm: geometry collision mesh filename=package://cmr_arm_sim/meshes/lower_arm.stl scale=0.1 0.1 0.1; visual mesh filename=package://cmr_arm_sim/meshes/lower_arm.stl scale=0.1 0.1 0.1
- link shoulder: geometry collision mesh filename=package://cmr_arm_sim/meshes/shoulder.stl scale=0.1 0.1 0.1; visual mesh filename=package://cmr_arm_sim/meshes/shoulder.stl scale=0.1 0.1 0.1
- link upper_arm: geometry collision mesh filename=package://cmr_arm_sim/meshes/upper_arm.stl scale=0.1 0.1 0.1; visual mesh filename=package://cmr_arm_sim/meshes/upper_arm.stl scale=0.1 0.1 0.1
- link wrist_rotate: geometry collision mesh filename=package://cmr_arm_sim/meshes/wrist_rotate.stl scale=0.1 0.1 0.1; visual mesh filename=package://cmr_arm_sim/meshes/wrist_rotate.stl scale=0.1 0.1 0.1
- link wrist_twist_rotate: geometry collision mesh filename=package://cmr_arm_sim/meshes/wrist_twist_rotate.stl scale=0.1 0.1 0.1; visual mesh filename=package://cmr_arm_sim/meshes/wrist_twist_rotate.stl scale=0.1 0.1 0.1
Joints:
- joint elbow_joint: origin xyz=0 -14.425 0 rpy=0 0 0 -> xyz=0 -1.4425 0 rpy=0 0 0
- joint shoulder_joint: origin xyz=0 0 3.61 rpy=0 0 0 -> xyz=0 -0.044 .361 rpy=0 0 0
- joint wrist_rotate: origin xyz=1.12 -14.425 0 rpy=0 0 0 -> xyz=.112 -1.4425 0 rpy=0 0 0
- joint wrist_rotate_two: origin xyz=-3.85 0 -4.2 rpy=0 0 0 -> xyz=-.385 0 -.42 rpy=0 0 0
- joint wrist_twist: origin xyz=0.0 -2 0.0508 rpy=0 0 0 -> xyz=0.0 -.2 0.00508 rpy=0 0 0

Commit message: rovernet arm

File: src/cmr_arm_sim/urdf/arm_2024.urdf (robot description, URDF)
Before this commit: robot Arm, 7 links, 6 joints
Links:
- link base_link: geometry visual mesh filename=package://cmr_arm_sim/meshes/base_link.stl scale=0.1 0.1 0.1
- link end_effector: geometry visual mesh filename=package://cmr_arm_sim/meshes/end_effector.stl scale=.0039 .0039 .0039
- link lower_arm: geometry visual mesh filename=package://cmr_arm_sim/meshes/lower_arm.stl scale=0.1 0.1 0.1
- link shoulder: geometry visual mesh filename=package://cmr_arm_sim/meshes/shoulder.stl scale=0.1 0.1 0.1
- link upper_arm: geometry visual mesh filename=package://cmr_arm_sim/meshes/upper_arm.stl scale=0.1 0.1 0.1
- link wrist_rotate: geometry visual mesh filename=package://cmr_arm_sim/meshes/wrist_rotate.stl scale=0.1 0.1 0.1
- link wrist_twist_rotate: geometry visual mesh filename=package://cmr_arm_sim/meshes/wrist_twist_rotate.stl scale=0.1 0.1 0.1

Commit message: cmr_arm_simulator

File: src/cmr_arm_sim/urdf/arm_2024.urdf (robot description, URDF)
Before this commit: robot Arm, 7 links, 6 joints
Joints:
- joint wrist_rotate_two: axis 0 1 0 -> 1 0 0

Commit message: Merging new MJBots comm board code, arm controller fix, new usb camera package (#77)
* Changed CCB specific code to use MJBOTS board

* Added new camera encoder code to view more cameras at once

* Decreased quality and made it so that terra can build outside of terra

File: src/cmr_arm_sim/urdf/arm_2024.urdf (robot description, URDF)
Before this commit: robot Arm, 7 links, 6 joints
Joints:
- joint wrist_rotate_two: axis 1 0 0 -> 0 1 0

Commit message: Updated URDF (first three joints are updated to new arm)

File: src/cmr_arm_sim/urdf/arm_2024.urdf (robot description, URDF)
Before this commit: robot Arm, 7 links, 6 joints
Links:
- link lower_arm: geometry visual mesh filename=package://cmr_arm_sim/meshes/lower_arm.stl scale=0.00375 0.00375 0.00375
- link shoulder: geometry visual mesh filename=package://cmr_arm_sim/meshes/shoulder.stl scale=0.00375 0.00375 0.00375
- link upper_arm: geometry visual mesh filename=package://cmr_arm_sim/meshes/upper_arm.stl scale=0.00375 0.00375 0.00375
- link wrist_rotate: geometry visual mesh filename=package://cmr_arm_sim/meshes/wrist_rotate.stl scale=0.00375 0.00375 0.00375
- link wrist_twist_rotate: geometry visual mesh filename=package://cmr_arm_sim/meshes/wrist_twist_rotate.stl scale=0.00375 0.00375 0.00375
Joints:
- joint base_joint: origin xyz=0.0 0.04335 0.0 rpy=0 0 0 -> xyz=0.0 0 1.1 rpy=0 0 0
- joint elbow_joint: child upper_arm -> wrist_rotate; origin xyz=0 -1.4425 0 rpy=0 0 0 -> xyz=0.09 -1.4425 0.015 rpy=0 0 0
- joint shoulder_joint: origin xyz=0 -0.044 .361 rpy=0 0 0 -> xyz=0 0 .251 rpy=-1.57079632679 0 0
- joint wrist_rotate: child wrist_rotate -> upper_arm; parent upper_arm -> wrist_rotate
- joint wrist_twist: parent wrist_rotate -> upper_arm

Commit message: new arm IK done

File: src/cmr_arm_sim/urdf/arm_2024.urdf (robot description, URDF)
Before this commit: robot Arm, 7 links, 6 joints
Joints:
- joint wrist_rotate: origin xyz=.112 -1.4425 0 rpy=0 0 0 -> xyz=0.21 0.01 0 rpy=0 0 0
- joint wrist_rotate_two: origin xyz=-.385 0 -.42 rpy=0 0 0 -> xyz=-0.205 -0.21 -0.01 rpy=0 0 0
- joint wrist_twist: axis 0 0 1 -> 1 0 0; origin xyz=0.0 -.2 0.00508 rpy=0 0 0 -> xyz=-0.03 -1.45 0.00508 rpy=0 0 0

Commit message: fixed arm

File: src/cmr_arm_sim/urdf/arm_2024.urdf (robot description, URDF)
Before this commit: robot Arm, 7 links, 6 joints
Joints:
- joint wrist_rotate_two: origin xyz=-0.205 -0.21 -0.01 rpy=0 0 0 -> xyz=-0.205 0.01 -0.01 rpy=0 0 0

Commit message: idk wtf this is

File: src/cmr_arm_sim/urdf/arm_2024.urdf (robot description, URDF)
Before this commit: robot Arm, 7 links, 6 joints
Joints:
- joint wrist_rotate_two: origin xyz=-0.205 0.01 -0.01 rpy=0 0 0 -> xyz=-0.205 -0.55 -0.01 rpy=0 0 0

Commit message: fix ishhaan

File: src/cmr_arm_sim/urdf/arm_2024.urdf (robot description, URDF)
Before this commit: robot Arm, 7 links, 6 joints
Joints:
- joint wrist_rotate_two: origin xyz=-.385 0 -.42 rpy=0 0 0 -> xyz=-0.205 -0.55 -0.01 rpy=0 0 0

Commit message: mostly working

File: src/cmr_arm_sim/urdf/arm_2024.urdf (robot description, URDF)
Before this commit: robot Arm, 7 links, 6 joints
Joints:
- joint wrist_rotate_two: origin xyz=-0.205 -0.55 -0.01 rpy=0 0 0 -> xyz=-0.205 -0.60 -0.01 rpy=0 0 0

Commit message: merge attempt 1 ready to test

File: src/cmr_arm_sim/urdf/arm_2024.urdf (robot description, URDF)
Before this commit: robot Arm, 7 links, 6 joints
Links:
- link lower_arm: geometry visual mesh filename=package://cmr_arm_sim/meshes/lower_arm.stl scale=0.00375 0.00375 0.00375
- link shoulder: geometry visual mesh filename=package://cmr_arm_sim/meshes/shoulder.stl scale=0.00375 0.00375 0.00375
- link upper_arm: geometry visual mesh filename=package://cmr_arm_sim/meshes/upper_arm.stl scale=0.00375 0.00375 0.00375
- link wrist_rotate: geometry visual mesh filename=package://cmr_arm_sim/meshes/wrist_rotate.stl scale=0.00375 0.00375 0.00375
- link wrist_twist_rotate: geometry visual mesh filename=package://cmr_arm_sim/meshes/wrist_twist_rotate.stl scale=0.00375 0.00375 0.00375
Joints:
- joint base_joint: origin xyz=0.0 0.04335 0.0 rpy=0 0 0 -> xyz=0.0 0 1.1 rpy=0 0 0
- joint elbow_joint: child upper_arm -> wrist_rotate; origin xyz=0 -1.4425 0 rpy=0 0 0 -> xyz=0.09 -1.4425 0.015 rpy=0 0 0
- joint shoulder_joint: origin xyz=0 -0.044 .361 rpy=0 0 0 -> xyz=0 0 .251 rpy=-1.57079632679 0 0
- joint wrist_rotate: child wrist_rotate -> upper_arm; origin xyz=.112 -1.4425 0 rpy=0 0 0 -> xyz=0.21 0.01 0 rpy=0 0 0; parent upper_arm -> wrist_rotate
- joint wrist_rotate_two: origin xyz=-.385 0 -.42 rpy=0 0 0 -> xyz=-0.205 -0.55 -0.01 rpy=0 0 0
- joint wrist_twist: axis 0 0 1 -> 1 0 0; origin xyz=0.0 -.2 0.00508 rpy=0 0 0 -> xyz=-0.03 -1.45 0.00508 rpy=0 0 0; parent wrist_rotate -> upper_arm
